File: hardware/pod_board/leds.kicad_sch (KiCad schematic)
At the start: 6 parts

Commit message: PCBs routed, labelled and ready to order: Rev 1 fabrication files and buy list
Both boards placed, routed and finished by script (hardware/gen): layout.sh places
(placement.py, with silkscreen names for every terminal, port, header and button),
route.sh routes with Freerouting inside rule areas and net classes from the layout
guide and keeps a board only with 0 DRC errors, 0 unconnected and exact schematic
parity, routespec.sh checks what the DRC cannot (planes, crystal, converter loop,
IPC-2221 widths), finish.sh adds the bottom-silkscreen identification and writes
the fabrication files (gerbers, drill, BOM, positions) only when the DRC passes.

- Pod 70 x 53 mm, 4 layers: In1 solid GND, In2 +3V3, 530 teardrops; no DRC warnings.
- Power 95 x 66 mm, 2 layers, 2 oz: 10 A rail as a zone, converter re-placed (switch
  node 16 mm, feedback 7 mm, no vias; was 78 mm and 40 mm), 328 teardrops.
- Screw terminals turned to open outward; RESET/BOOT side-push on the pod's left
  edge; USB-C footprint with a 3D model (GCT USB4105).
- Pod J2 now the Adafruit 4754's JP1 row pin for pin (the old order shorted its
  3.3 V output to ground); IMU reset on a new J8; HC-05 header fed 5 V.
- Buy list per footprint and module connections in bill-of-materials.md section 10.
- LAYOUT_GUIDE rewritten as how the boards were routed and how to review them;
  decisions, progress log and BUILD_GUIDE updated; power box follows the wider board.
Changed lines of the file:
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@@
 		(instances
 			(project "pod_board"
-				(path "/e1d1b1a6-cd0d-43ea-aa8d-30188448a190/8257df16-6369-4482-9d33-5388bbdbe70c"
+				(path "/f99c05c8-c1d8-4726-947c-3aab174eb82c/d56d8d79-a2c9-415f-97d8-2dc7d3b339ac"
 					(reference "R31")
 					(unit 1)
@@
 		(instances
 			(project "pod_board"
-				(path "/e1d1b1a6-cd0d-43ea-aa8d-30188448a190/8257df16-6369-4482-9d33-5388bbdbe70c"
+				(path "/f99c05c8-c1d8-4726-947c-3aab174eb82c/d56d8d79-a2c9-415f-97d8-2dc7d3b339ac"
 					(reference "D4")
 					(unit 1)
@@
 		(instances
 			(project "pod_board"
-				(path "/e1d1b1a6-cd0d-43ea-aa8d-30188448a190/8257df16-6369-4482-9d33-5388bbdbe70c"
+				(path "/f99c05c8-c1d8-4726-947c-3aab174eb82c/d56d8d79-a2c9-415f-97d8-2dc7d3b339ac"
 					(reference "R32")
 					(unit 1)
@@
 		(instances
 			(project "pod_board"
-				(path "/e1d1b1a6-cd0d-43ea-aa8d-30188448a190/8257df16-6369-4482-9d33-5388bbdbe70c"
+				(path "/f99c05c8-c1d8-4726-947c-3aab174eb82c/d56d8d79-a2c9-415f-97d8-2dc7d3b339ac"
 					(reference "D5")
 					(unit 1)
@@
 		(instances
 			(project "pod_board"
-				(path "/e1d1b1a6-cd0d-43ea-aa8d-30188448a190/8257df16-6369-4482-9d33-5388bbdbe70c"
+				(path "/f99c05c8-c1d8-4726-947c-3aab174eb82c/d56d8d79-a2c9-415f-97d8-2dc7d3b339ac"
 					(reference "R33")
 					(unit 1)
@@
 		(instances
 			(project "pod_board"
-				(path "/e1d1b1a6-cd0d-43ea-aa8d-30188448a190/8257df16-6369-4482-9d33-5388bbdbe70c"
+				(path "/f99c05c8-c1d8-4726-947c-3aab174eb82c/d56d8d79-a2c9-415f-97d8-2dc7d3b339ac"
 					(reference "D6")
 					(unit 1)
@@
 		(on_board yes)
 		(dnp no)
-		(property "Reference" "#PWR056"
+		(property "Reference" "#PWR055"
 			(at 121.92 85.09 0)
 			(hide yes)
@@
 		(instances
 			(project "pod_board"
-				(path "/e1d1b1a6-cd0d-43ea-aa8d-30188448a190/8257df16-6369-4482-9d33-5388bbdbe70c"
-					(reference "#PWR056")
+				(path "/f99c05c8-c1d8-4726-947c-3aab174eb82c/d56d8d79-a2c9-415f-97d8-2dc7d3b339ac"
+					(reference "#PWR055")
 					(unit 1)
 				)
@@
 		(on_board yes)
 		(dnp no)
-		(property "Reference" "#PWR057"
+		(property "Reference" "#PWR056"
 			(at 121.92 110.49 0)
 			(hide yes)
@@
 		(instances
 			(project "pod_board"
-				(path "/e1d1b1a6-cd0d-43ea-aa8d-30188448a190/8257df16-6369-4482-9d33-5388bbdbe70c"
-					(reference "#PWR057")
+				(path "/f99c05c8-c1d8-4726-947c-3aab174eb82c/d56d8d79-a2c9-415f-97d8-2dc7d3b339ac"
+					(reference "#PWR056")
 					(unit 1)
 				)
@@
 		(on_board yes)
 		(dnp no)
-		(property "Reference" "#PWR058"
+		(property "Reference" "#PWR057"
 			(at 121.92 135.89 0)
 			(hide yes)
@@
 		(instances
 			(project "pod_board"
-				(path "/e1d1b1a6-cd0d-43ea-aa8d-30188448a190/8257df16-6369-4482-9d33-5388bbdbe70c"
-					(reference "#PWR058")
+				(path "/f99c05c8-c1d8-4726-947c-3aab174eb82c/d56d8d79-a2c9-415f-97d8-2dc7d3b339ac"
+					(reference "#PWR057")
 					(unit 1)
 				)
@@
 	(wire
 		(pts
+			(xy 105.41 96.52)
+			(xy 106.68 96.52)
+		)
+		(stroke
+			(width 0)
+			(type default)
+		)
+	)
+	(wire
+		(pts
 			(xy 106.68 96.52)
 			(xy 121.92 96.52)
@@
 	(wire
 		(pts
-			(xy 106.68 96.52)
-			(xy 105.41 96.52)
-		)
-		(stroke
-			(width 0)
-			(type default)
-		)
-	)
-	(wire
-		(pts
 			(xy 121.92 96.52)
 			(xy 121.92 100.33)
@@
 	(wire
 		(pts
+			(xy 105.41 121.92)
+			(xy 106.68 121.92)
+		)
+		(stroke
+			(width 0)
+			(type default)
+		)
+	)
+	(wire
+		(pts
 			(xy 106.68 121.92)
 			(xy 121.92 121.92)
@@
 	(wire
 		(pts
-			(xy 105.41 121.92)
-			(xy 106.68 121.92)
-		)
-		(stroke
-			(width 0)
-			(type default)
-		)
-	)
-	(wire
-		(pts
-			(xy 121.92 71.12)
-			(xy 106.68 71.12)
-		)
-		(stroke
-			(width 0)
-			(type default)
-		)
-	)
-	(wire
-		(pts
 			(xy 105.41 71.12)
 			(xy 106.68 71.12)
@@
 	(wire
 		(pts
+			(xy 106.68 71.12)
+			(xy 121.92 71.12)
+		)
+		(stroke
+			(width 0)
+			(type default)
+		)
+	)
+	(wire
+		(pts
 			(xy 121.92 71.12)
 			(xy 121.92 74.93)
@@
 	(wire
 		(pts
+			(xy 30.48 121.92)
 			(xy 97.79 121.92)
-			(xy 30.48 121.92)
-		)
-		(stroke
+		)
+		(stroke
