File: hardware/pod_board/usb.kicad_sch (KiCad schematic)
At the start: 6 parts, among them J1 USB-C, U4 USBLC6-2SC6

Commit message: PCBs routed, labelled and ready to order: Rev 1 fabrication files and buy list
Both boards placed, routed and finished by script (hardware/gen): layout.sh places
(placement.py, with silkscreen names for every terminal, port, header and button),
route.sh routes with Freerouting inside rule areas and net classes from the layout
guide and keeps a board only with 0 DRC errors, 0 unconnected and exact schematic
parity, routespec.sh checks what the DRC cannot (planes, crystal, converter loop,
IPC-2221 widths), finish.sh adds the bottom-silkscreen identification and writes
the fabrication files (gerbers, drill, BOM, positions) only when the DRC passes.

- Pod 70 x 53 mm, 4 layers: In1 solid GND, In2 +3V3, 530 teardrops; no DRC warnings.
- Power 95 x 66 mm, 2 layers, 2 oz: 10 A rail as a zone, converter re-placed (switch
  node 16 mm, feedback 7 mm, no vias; was 78 mm and 40 mm), 328 teardrops.
- Screw terminals turned to open outward; RESET/BOOT side-push on the pod's left
  edge; USB-C footprint with a 3D model (GCT USB4105).
- Pod J2 now the Adafruit 4754's JP1 row pin for pin (the old order shorted its
  3.3 V output to ground); IMU reset on a new J8; HC-05 header fed 5 V.
- Buy list per footprint and module connections in bill-of-materials.md section 10.
- LAYOUT_GUIDE rewritten as how the boards were routed and how to review them;
  decisions, progress log and BUILD_GUIDE updated; power box follows the wider board.
Parts:
- J1: footprint Connector_USB:USB_C_Receptacle_HRO_TYPE-C-31-M-12 -> Connector_USB:USB_C_Receptacle_GCT_USB4105-xx-A_16P_TopMnt_Horizontal
