File: hardware/power_board/cable.kicad_sch (KiCad schematic)
At the start: 1 part, among them J1 DB-25 to pod

Commit message: PCBs routed, labelled and ready to order: Rev 1 fabrication files and buy list
Both boards placed, routed and finished by script (hardware/gen): layout.sh places
(placement.py, with silkscreen names for every terminal, port, header and button),
route.sh routes with Freerouting inside rule areas and net classes from the layout
guide and keeps a board only with 0 DRC errors, 0 unconnected and exact schematic
parity, routespec.sh checks what the DRC cannot (planes, crystal, converter loop,
IPC-2221 widths), finish.sh adds the bottom-silkscreen identification and writes
the fabrication files (gerbers, drill, BOM, positions) only when the DRC passes.

- Pod 70 x 53 mm, 4 layers: In1 solid GND, In2 +3V3, 530 teardrops; no DRC warnings.
- Power 95 x 66 mm, 2 layers, 2 oz: 10 A rail as a zone, converter re-placed (switch
  node 16 mm, feedback 7 mm, no vias; was 78 mm and 40 mm), 328 teardrops.
- Screw terminals turned to open outward; RESET/BOOT side-push on the pod's left
  edge; USB-C footprint with a 3D model (GCT USB4105).
- Pod J2 now the Adafruit 4754's JP1 row pin for pin (the old order shorted its
  3.3 V output to ground); IMU reset on a new J8; HC-05 header fed 5 V.
- Buy list per footprint and module connections in bill-of-materials.md section 10.
- LAYOUT_GUIDE rewritten as how the boards were routed and how to review them;
  decisions, progress log and BUILD_GUIDE updated; power box follows the wider board.
Changed lines of the file:
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@@
 		(instances
 			(project "power_board"
-				(path "/244ac675-494c-4e27-8819-02215b480bc3/657b2369-8e36-47b4-85e3-65704dfa8b5b"
+				(path "/c794bf93-11d2-4d5c-a02b-6bb49c306097/7d782f74-e0d0-4329-ba3e-d50e8edb7165"
 					(reference "J1")
 					(unit 1)
@@
 		(instances
 			(project "power_board"
-				(path "/244ac675-494c-4e27-8819-02215b480bc3/657b2369-8e36-47b4-85e3-65704dfa8b5b"
+				(path "/c794bf93-11d2-4d5c-a02b-6bb49c306097/7d782f74-e0d0-4329-ba3e-d50e8edb7165"
 					(reference "#PWR084")
 					(unit 1)
@@
 		(instances
 			(project "power_board"
-				(path "/244ac675-494c-4e27-8819-02215b480bc3/657b2369-8e36-47b4-85e3-65704dfa8b5b"
+				(path "/c794bf93-11d2-4d5c-a02b-6bb49c306097/7d782f74-e0d0-4329-ba3e-d50e8edb7165"
 					(reference "#PWR085")
 					(unit 1)
@@
 		(instances
 			(project "power_board"
-				(path "/244ac675-494c-4e27-8819-02215b480bc3/657b2369-8e36-47b4-85e3-65704dfa8b5b"
+				(path "/c794bf93-11d2-4d5c-a02b-6bb49c306097/7d782f74-e0d0-4329-ba3e-d50e8edb7165"
 					(reference "#PWR086")
 					(unit 1)
@@
 		(instances
 			(project "power_board"
-				(path "/244ac675-494c-4e27-8819-02215b480bc3/657b2369-8e36-47b4-85e3-65704dfa8b5b"
+				(path "/c794bf93-11d2-4d5c-a02b-6bb49c306097/7d782f74-e0d0-4329-ba3e-d50e8edb7165"
 					(reference "#PWR087")
 					(unit 1)
@@
 		(instances
 			(project "power_board"
-				(path "/244ac675-494c-4e27-8819-02215b480bc3/657b2369-8e36-47b4-85e3-65704dfa8b5b"
+				(path "/c794bf93-11d2-4d5c-a02b-6bb49c306097/7d782f74-e0d0-4329-ba3e-d50e8edb7165"
 					(reference "#PWR088")
 					(unit 1)
@@
 		(instances
 			(project "power_board"
-				(path "/244ac675-494c-4e27-8819-02215b480bc3/657b2369-8e36-47b4-85e3-65704dfa8b5b"
+				(path "/c794bf93-11d2-4d5c-a02b-6bb49c306097/7d782f74-e0d0-4329-ba3e-d50e8edb7165"
 					(reference "#PWR089")
 					(unit 1)
@@
 	(wire
 		(pts
+			(xy 73.66 147.32)
 			(xy 177.8 147.32)
-			(xy 73.66 147.32)
-		)
-		(stroke
-			(width 0)
-			(type default)
-		)
-	)
-	(wire
-		(pts
+		)
+		(stroke
+			(width 0)
+			(type default)
+		)
+	)
+	(wire
+		(pts
+			(xy 73.66 132.08)
 			(xy 177.8 132.08)
-			(xy 73.66 132.08)
 		)
 		(stroke
@@
 	(wire
 		(pts
+			(xy 73.66 114.3)
 			(xy 177.8 114.3)
-			(xy 73.66 114.3)
 		)
 		(stroke
@@
 	(wire
 		(pts
+			(xy 73.66 106.68)
 			(xy 177.8 106.68)
-			(xy 73.66 106.68)
-		)
-		(stroke
-			(width 0)
-			(type default)
-		)
-	)
-	(wire
-		(pts
+		)
+		(stroke
+			(width 0)
+			(type default)
+		)
+	)
+	(wire
+		(pts
+			(xy 73.66 124.46)
 			(xy 177.8 124.46)
-			(xy 73.66 124.46)
 		)
 		(stroke
@@
 	(wire
 		(pts
+			(xy 73.66 127.0)
 			(xy 177.8 127.0)
-			(xy 73.66 127.0)
-		)
-		(stroke
-			(width 0)
-			(type default)
-		)
-	)
-	(wire
-		(pts
+		)
+		(stroke
+			(width 0)
+			(type default)
+		)
+	)
+	(wire
+		(pts
+			(xy 73.66 109.22)
 			(xy 177.8 109.22)
-			(xy 73.66 109.22)
 		)
 		(stroke
@@
 	(wire
 		(pts
+			(xy 73.66 86.36)
+			(xy 74.93 86.36)
+		)
+		(stroke
+			(width 0)
+			(type default)
+		)
+	)
+	(wire
+		(pts
+			(xy 73.66 91.44)
+			(xy 74.93 91.44)
+		)
+		(stroke
+			(width 0)
+			(type default)
+		)
+	)
+	(wire
+		(pts
+			(xy 74.93 86.36)
+			(xy 74.93 91.44)
+		)
+		(stroke
+			(width 0)
+			(type default)
+		)
+	)
+	(wire
+		(pts
 			(xy 74.93 86.36)
 			(xy 177.8 86.36)
 		)
 		(stroke
-			(width 0)
-			(type default)
-		)
-	)
-	(wire
-		(pts
-			(xy 74.93 86.36)
-			(xy 74.93 91.44)
-		)
-		(stroke
-			(width 0)
-			(type default)
-		)
-	)
-	(wire
-		(pts
-			(xy 73.66 86.36)
-			(xy 74.93 86.36)
-		)
-		(stroke
-			(width 0)
-			(type default)
-		)
-	)
-	(wire
-		(pts
-			(xy 73.66 91.44)
-			(xy 74.93 91.44)
-		)
-		(stroke
