File: hardware/power_board/can.kicad_sch (KiCad schematic)
At the start: 6 parts, among them J11 OBD-II lead, U4 SN65HVD230

Commit message: Pod board schematic redrawn as wired sheets; duplicate references fixed
pod_board_drawing.py draws six sheets around an MCU sheet under a block
diagram; check.sh now compares both boards' drawn and label-only netlists.
kisheet.py: stacked pins, PWR_FLAGs on signal nets, column hints for
crossing-free fan-ins, nets drawn in pieces joined by name, and visible
rail names on power symbols.

R31-R33 were used twice on the pod board, which KiCad's ERC does not
report; the netlist merged each pair. Cable parts now start at R40/C40,
generate.py rejects duplicate references and check_nets.py fails on a pin
in two nets. check_nets.py also drops the sheet path from net names.
Changed lines of the file:
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@@
 		(instances
 			(project "power_board"
-				(path "/3aef661e-32a5-4098-b535-e9581569514f/a5ab398b-6c59-4377-bef7-f1aff6ada48c"
+				(path "/244ac675-494c-4e27-8819-02215b480bc3/a498b140-102b-436f-aa23-4911f5714cb2"
 					(reference "R59")
 					(unit 1)
@@
 		(instances
 			(project "power_board"
-				(path "/3aef661e-32a5-4098-b535-e9581569514f/a5ab398b-6c59-4377-bef7-f1aff6ada48c"
+				(path "/244ac675-494c-4e27-8819-02215b480bc3/a498b140-102b-436f-aa23-4911f5714cb2"
 					(reference "R60")
 					(unit 1)
@@
 		(instances
 			(project "power_board"
-				(path "/3aef661e-32a5-4098-b535-e9581569514f/a5ab398b-6c59-4377-bef7-f1aff6ada48c"
+				(path "/244ac675-494c-4e27-8819-02215b480bc3/a498b140-102b-436f-aa23-4911f5714cb2"
 					(reference "U4")
 					(unit 1)
@@
 		(instances
 			(project "power_board"
-				(path "/3aef661e-32a5-4098-b535-e9581569514f/a5ab398b-6c59-4377-bef7-f1aff6ada48c"
+				(path "/244ac675-494c-4e27-8819-02215b480bc3/a498b140-102b-436f-aa23-4911f5714cb2"
 					(reference "C32")
 					(unit 1)
@@
 		(instances
 			(project "power_board"
-				(path "/3aef661e-32a5-4098-b535-e9581569514f/a5ab398b-6c59-4377-bef7-f1aff6ada48c"
+				(path "/244ac675-494c-4e27-8819-02215b480bc3/a498b140-102b-436f-aa23-4911f5714cb2"
 					(reference "D20")
 					(unit 1)
@@
 		(instances
 			(project "power_board"
-				(path "/3aef661e-32a5-4098-b535-e9581569514f/a5ab398b-6c59-4377-bef7-f1aff6ada48c"
+				(path "/244ac675-494c-4e27-8819-02215b480bc3/a498b140-102b-436f-aa23-4911f5714cb2"
 					(reference "J11")
 					(unit 1)
@@
 		)
 		(property "Value" "+3V3"
-			(at 76.2 82.55 0)
-			(hide yes)
-			(effects
-				(font
-					(size 1.0 1.0)
+			(at 76.2 78.95 0)
+			(effects
+				(font
+					(size 1.27 1.27)
 				)
 			)
@@
 		(instances
 			(project "power_board"
-				(path "/3aef661e-32a5-4098-b535-e9581569514f/a5ab398b-6c59-4377-bef7-f1aff6ada48c"
+				(path "/244ac675-494c-4e27-8819-02215b480bc3/a498b140-102b-436f-aa23-4911f5714cb2"
 					(reference "#PWR064")
 					(unit 1)
@@
 		)
 		(property "Value" "+3V3"
-			(at 76.2 110.49 0)
-			(hide yes)
-			(effects
-				(font
-					(size 1.0 1.0)
+			(at 76.2 106.89 0)
+			(effects
+				(font
+					(size 1.27 1.27)
 				)
 			)
@@
 		(instances
 			(project "power_board"
-				(path "/3aef661e-32a5-4098-b535-e9581569514f/a5ab398b-6c59-4377-bef7-f1aff6ada48c"
+				(path "/244ac675-494c-4e27-8819-02215b480bc3/a498b140-102b-436f-aa23-4911f5714cb2"
 					(reference "#PWR065")
 					(unit 1)
@@
 		)
 		(property "Value" "GND"
-			(at 127.0 114.3 0)
-			(hide yes)
-			(effects
-				(font
-					(size 1.0 1.0)
+			(at 127.0 110.7 0)
+			(hide yes)
+			(effects
+				(font
+					(size 1.27 1.27)
 				)
 			)
@@
 		(instances
 			(project "power_board"
-				(path "/3aef661e-32a5-4098-b535-e9581569514f/a5ab398b-6c59-4377-bef7-f1aff6ada48c"
+				(path "/244ac675-494c-4e27-8819-02215b480bc3/a498b140-102b-436f-aa23-4911f5714cb2"
 					(reference "#PWR066")
 					(unit 1)
@@
 		)
 		(property "Value" "+3V3"
-			(at 127.0 91.44 0)
-			(hide yes)
-			(effects
-				(font
-					(size 1.0 1.0)
+			(at 127.0 87.84 0)
+			(effects
+				(font
+					(size 1.27 1.27)
 				)
 			)
@@
 		(instances
 			(project "power_board"
-				(path "/3aef661e-32a5-4098-b535-e9581569514f/a5ab398b-6c59-4377-bef7-f1aff6ada48c"
+				(path "/244ac675-494c-4e27-8819-02215b480bc3/a498b140-102b-436f-aa23-4911f5714cb2"
 					(reference "#PWR067")
 					(unit 1)
@@
 		)
 		(property "Value" "+3V3"
-			(at 106.68 69.85 0)
-			(hide yes)
-			(effects
-				(font
-					(size 1.0 1.0)
+			(at 106.68 66.25 0)
+			(effects
+				(font
+					(size 1.27 1.27)
 				)
 			)
@@
 		(instances
 			(project "power_board"
-				(path "/3aef661e-32a5-4098-b535-e9581569514f/a5ab398b-6c59-4377-bef7-f1aff6ada48c"
+				(path "/244ac675-494c-4e27-8819-02215b480bc3/a498b140-102b-436f-aa23-4911f5714cb2"
 					(reference "#PWR068")
 					(unit 1)
@@
 		)
 		(property "Value" "GND"
-			(at 106.68 82.55 0)
-			(hide yes)
-			(effects
-				(font
-					(size 1.0 1.0)
+			(at 106.68 78.95 0)
+			(hide yes)
+			(effects
+				(font
+					(size 1.27 1.27)
 				)
 			)
@@
 		(instances
 			(project "power_board"
-				(path "/3aef661e-32a5-4098-b535-e9581569514f/a5ab398b-6c59-4377-bef7-f1aff6ada48c"
+				(path "/244ac675-494c-4e27-8819-02215b480bc3/a498b140-102b-436f-aa23-4911f5714cb2"
 					(reference "#PWR069")
 					(unit 1)
@@
 		)
 		(property "Value" "GND"
-			(at 157.48 127.0 0)
-			(hide yes)
-			(effects
-				(font
-					(size 1.0 1.0)
+			(at 157.48 123.4 0)
+			(hide yes)
+			(effects
+				(font
+					(size 1.27 1.27)
 				)
 			)
@@
 		(instances
 			(project "power_board"
-				(path "/3aef661e-32a5-4098-b535-e9581569514f/a5ab398b-6c59-4377-bef7-f1aff6ada48c"
+				(path "/244ac675-494c-4e27-8819-02215b480bc3/a498b140-102b-436f-aa23-4911f5714cb2"
 					(reference "#PWR070")
 					(unit 1)
@@
 		)
 		(property "Value" "GND"
-			(at 195.58 109.22 0)
-			(hide yes)
-			(effects
-				(font
-					(size 1.0 1.0)
+			(at 195.58 105.62 0)
+			(hide yes)
+			(effects
+				(font
+					(size 1.27 1.27)
 				)
 			)
@@
 		(instances
 			(project "power_board"
-				(path "/3aef661e-32a5-4098-b535-e9581569514f/a5ab398b-6c59-4377-bef7-f1aff6ada48c"
+				(path "/244ac675-494c-4e27-8819-02215b480bc3/a498b140-102b-436f-aa23-4911f5714cb2"
 					(reference "#PWR071")
 					(unit 1)

Commit message: PCBs routed, labelled and ready to order: Rev 1 fabrication files and buy list
Both boards placed, routed and finished by script (hardware/gen): layout.sh places
(placement.py, with silkscreen names for every terminal, port, header and button),
route.sh routes with Freerouting inside rule areas and net classes from the layout
guide and keeps a board only with 0 DRC errors, 0 unconnected and exact schematic
parity, routespec.sh checks what the DRC cannot (planes, crystal, converter loop,
IPC-2221 widths), finish.sh adds the bottom-silkscreen identification and writes
the fabrication files (gerbers, drill, BOM, positions) only when the DRC passes.

- Pod 70 x 53 mm, 4 layers: In1 solid GND, In2 +3V3, 530 teardrops; no DRC warnings.
- Power 95 x 66 mm, 2 layers, 2 oz: 10 A rail as a zone, converter re-placed (switch
  node 16 mm, feedback 7 mm, no vias; was 78 mm and 40 mm), 328 teardrops.
- Screw terminals turned to open outward; RESET/BOOT side-push on the pod's left
  edge; USB-C footprint with a 3D model (GCT USB4105).
- Pod J2 now the Adafruit 4754's JP1 row pin for pin (the old order shorted its
  3.3 V output to ground); IMU reset on a new J8; HC-05 header fed 5 V.
- Buy list per footprint and module connections in bill-of-materials.md section 10.
- LAYOUT_GUIDE rewritten as how the boards were routed and how to review them;
  decisions, progress log and BUILD_GUIDE updated; power box follows the wider board.
Changed lines of the file:
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@@
 		(instances
 			(project "power_board"
-				(path "/244ac675-494c-4e27-8819-02215b480bc3/a498b140-102b-436f-aa23-4911f5714cb2"
+				(path "/c794bf93-11d2-4d5c-a02b-6bb49c306097/00abe930-5ad3-4689-aa2b-99f9f99ed3cd"
 					(reference "R59")
 					(unit 1)
@@
 		(instances
 			(project "power_board"
-				(path "/244ac675-494c-4e27-8819-02215b480bc3/a498b140-102b-436f-aa23-4911f5714cb2"
+				(path "/c794bf93-11d2-4d5c-a02b-6bb49c306097/00abe930-5ad3-4689-aa2b-99f9f99ed3cd"
 					(reference "R60")
 					(unit 1)
@@
 		(instances
 			(project "power_board"
-				(path "/244ac675-494c-4e27-8819-02215b480bc3/a498b140-102b-436f-aa23-4911f5714cb2"
+				(path "/c794bf93-11d2-4d5c-a02b-6bb49c306097/00abe930-5ad3-4689-aa2b-99f9f99ed3cd"
 					(reference "U4")
 					(unit 1)
@@
 		(instances
 			(project "power_board"
-				(path "/244ac675-494c-4e27-8819-02215b480bc3/a498b140-102b-436f-aa23-4911f5714cb2"
+				(path "/c794bf93-11d2-4d5c-a02b-6bb49c306097/00abe930-5ad3-4689-aa2b-99f9f99ed3cd"
 					(reference "C32")
 					(unit 1)
@@
 		(instances
 			(project "power_board"
-				(path "/244ac675-494c-4e27-8819-02215b480bc3/a498b140-102b-436f-aa23-4911f5714cb2"
+				(path "/c794bf93-11d2-4d5c-a02b-6bb49c306097/00abe930-5ad3-4689-aa2b-99f9f99ed3cd"
 					(reference "D20")
 					(unit 1)
@@
 		(instances
 			(project "power_board"
-				(path "/244ac675-494c-4e27-8819-02215b480bc3/a498b140-102b-436f-aa23-4911f5714cb2"
+				(path "/c794bf93-11d2-4d5c-a02b-6bb49c306097/00abe930-5ad3-4689-aa2b-99f9f99ed3cd"
 					(reference "J11")
 					(unit 1)
@@
 		(instances
 			(project "power_board"
-				(path "/244ac675-494c-4e27-8819-02215b480bc3/a498b140-102b-436f-aa23-4911f5714cb2"
+				(path "/c794bf93-11d2-4d5c-a02b-6bb49c306097/00abe930-5ad3-4689-aa2b-99f9f99ed3cd"
 					(reference "#PWR064")
 					(unit 1)
@@
 		(instances
 			(project "power_board"
-				(path "/244ac675-494c-4e27-8819-02215b480bc3/a498b140-102b-436f-aa23-4911f5714cb2"
+				(path "/c794bf93-11d2-4d5c-a02b-6bb49c306097/00abe930-5ad3-4689-aa2b-99f9f99ed3cd"
 					(reference "#PWR065")
 					(unit 1)
@@
 		(instances
 			(project "power_board"
-				(path "/244ac675-494c-4e27-8819-02215b480bc3/a498b140-102b-436f-aa23-4911f5714cb2"
+				(path "/c794bf93-11d2-4d5c-a02b-6bb49c306097/00abe930-5ad3-4689-aa2b-99f9f99ed3cd"
 					(reference "#PWR066")
 					(unit 1)
@@
 		(instances
 			(project "power_board"
-				(path "/244ac675-494c-4e27-8819-02215b480bc3/a498b140-102b-436f-aa23-4911f5714cb2"
+				(path "/c794bf93-11d2-4d5c-a02b-6bb49c306097/00abe930-5ad3-4689-aa2b-99f9f99ed3cd"
 					(reference "#PWR067")
 					(unit 1)
@@
 		(instances
 			(project "power_board"
-				(path "/244ac675-494c-4e27-8819-02215b480bc3/a498b140-102b-436f-aa23-4911f5714cb2"
+				(path "/c794bf93-11d2-4d5c-a02b-6bb49c306097/00abe930-5ad3-4689-aa2b-99f9f99ed3cd"
 					(reference "#PWR068")
 					(unit 1)
@@
 		(instances
 			(project "power_board"
-				(path "/244ac675-494c-4e27-8819-02215b480bc3/a498b140-102b-436f-aa23-4911f5714cb2"
+				(path "/c794bf93-11d2-4d5c-a02b-6bb49c306097/00abe930-5ad3-4689-aa2b-99f9f99ed3cd"
 					(reference "#PWR069")
 					(unit 1)
@@
 		(instances
 			(project "power_board"
-				(path "/244ac675-494c-4e27-8819-02215b480bc3/a498b140-102b-436f-aa23-4911f5714cb2"
+				(path "/c794bf93-11d2-4d5c-a02b-6bb49c306097/00abe930-5ad3-4689-aa2b-99f9f99ed3cd"
 					(reference "#PWR070")
 					(unit 1)
@@
 		(instances
 			(project "power_board"
-				(path "/244ac675-494c-4e27-8819-02215b480bc3/a498b140-102b-436f-aa23-4911f5714cb2"
+				(path "/c794bf93-11d2-4d5c-a02b-6bb49c306097/00abe930-5ad3-4689-aa2b-99f9f99ed3cd"
 					(reference "#PWR071")
 					(unit 1)
@@
 	(wire
 		(pts
+			(xy 137.16 104.14)
+			(xy 138.43 104.14)
+		)
+		(stroke
+			(width 0)
+			(type default)
+		)
+	)
+	(wire
+		(pts
+			(xy 138.43 104.14)
+			(xy 160.02 104.14)
+		)
+		(stroke
+			(width 0)
+			(type default)
+		)
+	)
+	(wire
+		(pts
+			(xy 160.02 104.14)
+			(xy 160.02 114.3)
+		)
+		(stroke
+			(width 0)
+			(type default)
+		)
+	)
+	(wire
+		(pts
 			(xy 160.02 104.14)
 			(xy 198.12 104.14)
-		)
-		(stroke
-			(width 0)
-			(type default)
-		)
-	)
-	(wire
-		(pts
-			(xy 138.43 104.14)
-			(xy 160.02 104.14)
-		)
-		(stroke
-			(width 0)
-			(type default)
-		)
-	)
-	(wire
-		(pts
-			(xy 160.02 104.14)
-			(xy 160.02 114.3)
-		)
-		(stroke
-			(width 0)
-			(type default)
-		)
-	)
-	(wire
-		(pts
-			(xy 137.16 104.14)
-			(xy 138.43 104.14)
 		)
 		(stroke
@@
 	(wire
 		(pts
+			(xy 137.16 101.6)
+			(xy 138.43 101.6)
+		)
+		(stroke
+			(width 0)
+			(type default)
+		)
+	)
+	(wire
+		(pts
+			(xy 138.43 101.6)
+			(xy 154.94 101.6)
+		)
+		(stroke
+			(width 0)
+			(type default)
+		)
+	)
+	(wire
+		(pts
 			(xy 154.94 101.6)
 			(xy 154.94 114.3)
@@
 			(xy 154.94 101.6)
 			(xy 198.12 101.6)
-		)
-		(stroke
-			(width 0)
-			(type default)
-		)
-	)
-	(wire
-		(pts
-			(xy 154.94 101.6)
-			(xy 138.43 101.6)
-		)
-		(stroke
-			(width 0)
-			(type default)
-		)
-	)
-	(wire
-		(pts
-			(xy 138.43 101.6)
-			(xy 137.16 101.6)
 		)
 		(stroke
@@
 	(wire
 		(pts
+			(xy 30.48 99.06)
+			(xy 76.2 99.06)
+		)
+		(stroke
+			(width 0)
+			(type default)
+		)
+	)
+	(wire
+		(pts
+			(xy 76.2 92.71)
+			(xy 76.2 99.06)
+		)
+		(stroke
+			(width 0)
+			(type default)
+		)
+	)
+	(wire
+		(pts
+			(xy 76.2 99.06)
 			(xy 116.84 99.06)
-			(xy 76.2 99.06)
-		)
-		(stroke
-			(width 0)
-			(type default)
-		)
-	)
-	(wire
-		(pts
-			(xy 76.2 99.06)
-			(xy 30.48 99.06)
-		)
-		(stroke
-			(width 0)
-			(type default)
-		)
-	)
-	(wire
-		(pts
-			(xy 76.2 99.06)
-			(xy 76.2 92.71)
 		)
 		(stroke
@@
 	(wire
 		(pts
+			(xy 76.2 120.65)
+			(xy 76.2 121.92)
+		)
+		(stroke
+			(width 0)
+			(type default)
+		)
+	)
+	(wire
+		(pts
+			(xy 76.2 121.92)
+			(xy 76.2 127.0)
+		)
+		(stroke
+			(width 0)
+			(type default)
+		)
+	)
+	(wire
+		(pts
+			(xy 76.2 121.92)
+			(xy 82.55 121.92)
+		)
+		(stroke
+			(width 0)
+			(type default)
+		)
+	)
+	(wire
+		(pts
+			(xy 82.55 106.68)
+			(xy 82.55 121.92)
+		)
+		(stroke
+			(width 0)
+			(type default)
+		)
+	)
+	(wire
+		(pts
 			(xy 82.55 106.68)
 			(xy 116.84 106.68)
 		)
 		(stroke
-			(width 0)
-			(type default)
-		)
-	)
-	(wire
-		(pts
-			(xy 82.55 106.68)
-			(xy 82.55 121.92)
-		)
-		(stroke
-			(width 0)
-			(type default)
-		)
-	)
-	(wire
-		(pts
-			(xy 76.2 127.0)
-			(xy 76.2 121.92)
-		)
-		(stroke
-			(width 0)
-			(type default)
-		)
-	)
-	(wire
-		(pts
-			(xy 76.2 121.92)
-			(xy 82.55 121.92)
-		)
-		(stroke
-			(width 0)
-			(type default)
-		)
-	)
-	(wire
-		(pts
-			(xy 76.2 120.65)
-			(xy 76.2 121.92)
-		)
-		(stroke
