File: hardware/power_board/power_board.kicad_sch (KiCad schematic)
At the start: 82 parts, among them J1 DB-25 to pod, J10 Brake-light switch, J11 OBD-II lead, J12 Bench: HX711, J13 BTS7960 module, J14 ACS712 module, J2 12 V ACC in, J3 LiDAR 12 V out, J4 Relay coils, J5 Actuator 12 V from kill relay, J6 BTS7960 B+ / B-, J7 Cable magnet, J8 Kill relay coil feed, J9 E-stop sense contact, Q2 AO3400A, Q3 AO3400A, Q4 AO3400A, Q5 AO3400A, Q6 AO3400A, Q7 AO3400A, Q8 2N7002, U1 TPS54360DDA, U2 AP2112K-3.3, U3 74HCT244, U4 SN65HVD230, U5 PC817

Commit message: Power board schematic redrawn as wired sheets under a block diagram
kisheet.py writes hierarchical KiCad sheets with parts placed by hand and
wires routed between pins; power_board_drawing.py lays out eight function
sheets and the root block diagram. check.sh also builds the label-only
version and requires identical netlists (compare_nets.py).

Fixes check_nets.py reading no components from KiCad 10 netlists, which
made the footprint check pass with nothing to check.
Parts:
- removed C20: 47u 63V, Capacitor_THT:CP_Radial_D8.0mm_P3.50mm, symbol Device:C_Polarized
- removed C21, C22: 2.2u 100V, Capacitor_SMD:C_1210_3225Metric, symbol Device:C
- removed C23, C31, C32: 100n, Capacitor_SMD:C_0805_2012Metric, symbol Device:C
- removed C24, C25: 47u, Capacitor_SMD:C_1210_3225Metric, symbol Device:C
- removed C26: 6800p, Capacitor_SMD:C_0805_2012Metric, symbol Device:C
- removed C27: 39p, Capacitor_SMD:C_0805_2012Metric, symbol Device:C
- removed C28, C29, C30: 10u, Capacitor_SMD:C_1206_3216Metric, symbol Device:C
- removed D10: SMCJ24CA, Diode_SMD:D_SMC, symbol Device:D_TVS
- removed D11, D13: B560C, Diode_SMD:D_SMC, symbol Device:D_Schottky
- removed D12: green, LED_SMD:LED_0805_2012Metric, symbol Device:LED
- removed D14, D15, D16, D17, D18, D19: SS14, Diode_SMD:D_SMA, symbol Device:D_Schottky
- removed D20: NUP2105L, Package_TO_SOT_SMD:SOT-23, symbol Power_Protection:NUP2105L
- removed D21: 1N4148W, Diode_SMD:D_SOD-123, symbol Device:D
- removed F1, F3: 3A, Fuse:Fuseholder_Blade_Mini_Keystone_3568, symbol Device:Fuse
- removed F2: 500mA, Fuse:Fuse_1206_3216Metric, symbol Device:Polyfuse
- removed H1, H2, H3, H4: M3, MountingHole:MountingHole_3.2mm_M3, symbol Mechanical:MountingHole
- removed J1: DB-25 to pod, Connector_Dsub:DSUB-25_Socket_Horizontal_P2.77x2.84mm_EdgePinOffset4.94mm_Housed_MountingHolesOffset4.94mm, symbol Connector:DB25_Socket_MountingHoles
- removed J10: Brake-light switch, TerminalBlock_Phoenix:TerminalBlock_Phoenix_MKDS-1,5-2-5.08_1x02_P5.08mm_Horizontal, symbol Connector:Screw_Terminal_01x02
- removed J11: OBD-II lead, TerminalBlock_Phoenix:TerminalBlock_Phoenix_MKDS-1,5-3-5.08_1x03_P5.08mm_Horizontal, symbol Connector:Screw_Terminal_01x03
- removed J12: Bench: HX711, Connector_PinHeader_2.54mm:PinHeader_1x04_P2.54mm_Vertical, symbol Connector_Generic:Conn_01x04
- removed J13: BTS7960 module, Connector_PinHeader_2.54mm:PinHeader_1x08_P2.54mm_Vertical, symbol Connector_Generic:Conn_01x08
- removed J14: ACS712 module, Connector_PinHeader_2.54mm:PinHeader_1x03_P2.54mm_Vertical, symbol Connector_Generic:Conn_01x03
- removed J2: 12 V ACC in, TerminalBlock_Phoenix:TerminalBlock_Phoenix_MKDS-1,5-2-5.08_1x02_P5.08mm_Horizontal, symbol Connector:Screw_Terminal_01x02
- removed J3: LiDAR 12 V out, TerminalBlock_Phoenix:TerminalBlock_Phoenix_MKDS-1,5-2-5.08_1x02_P5.08mm_Horizontal, symbol Connector:Screw_Terminal_01x02
- removed J4: Relay coils, TerminalBlock_Phoenix:TerminalBlock_Phoenix_MKDS-1,5-6-5.08_1x06_P5.08mm_Horizontal, symbol Connector:Screw_Terminal_01x06
- removed J5: Actuator 12 V from kill relay, TerminalBlock_Phoenix:TerminalBlock_Phoenix_MKDS-1,5-2-5.08_1x02_P5.08mm_Horizontal, symbol Connector:Screw_Terminal_01x02
- removed J6: BTS7960 B+ / B-, TerminalBlock_Phoenix:TerminalBlock_Phoenix_MKDS-1,5-2-5.08_1x02_P5.08mm_Horizontal, symbol Connector:Screw_Terminal_01x02
- removed J7: Cable magnet, TerminalBlock_Phoenix:TerminalBlock_Phoenix_MKDS-1,5-2-5.08_1x02_P5.08mm_Horizontal, symbol Connector:Screw_Terminal_01x02
- removed J8: Kill relay coil feed, TerminalBlock_Phoenix:TerminalBlock_Phoenix_MKDS-1,5-2-5.08_1x02_P5.08mm_Horizontal, symbol Connector:Screw_Terminal_01x02
- removed J9: E-stop sense contact, TerminalBlock_Phoenix:TerminalBlock_Phoenix_MKDS-1,5-2-5.08_1x02_P5.08mm_Horizontal, symbol Connector:Screw_Terminal_01x02
- removed L1: 8.2u, Inductor_SMD:L_Bourns_SRR1260, symbol Device:L
- removed Q2, Q3, Q4, Q5, Q6, Q7: AO3400A, Package_TO_SOT_SMD:SOT-23, symbol Transistor_FET:AO3400A
- removed Q8: 2N7002, Package_TO_SOT_SMD:SOT-23, symbol Transistor_FET:2N7002
- removed R40: 4.7k, Resistor_SMD:R_0805_2012Metric, symbol Device:R
- removed R41: 523k, Resistor_SMD:R_0805_2012Metric, symbol Device:R
- removed R42: 84.5k, Resistor_SMD:R_0805_2012Metric, symbol Device:R
- removed R43: 162k, Resistor_SMD:R_0805_2012Metric, symbol Device:R
- removed R44: 53.6k, Resistor_SMD:R_0805_2012Metric, symbol Device:R
- removed R45: 10.2k, Resistor_SMD:R_0805_2012Metric, symbol Device:R
- removed R46: 13.0k, Resistor_SMD:R_0805_2012Metric, symbol Device:R
- removed R47, R50, R51, R52, R53, R54, R55, R56, R57, R58, R59, R60, R61: 10k, Resistor_SMD:R_0805_2012Metric, symbol Device:R
- removed R48: 20k, Resistor_SMD:R_0805_2012Metric, symbol Device:R
- removed R62: 100k, Resistor_SMD:R_0805_2012Metric, symbol Device:R
- removed R63: 2.2k, Resistor_SMD:R_0805_2012Metric, symbol Device:R
- removed U1: TPS54360DDA, Package_SO:TI_SO-PowerPAD-8_ThermalVias, symbol Regulator_Switching:TPS54360DDA
- removed U2: AP2112K-3.3, Package_TO_SOT_SMD:SOT-23-5, symbol Regulator_Linear:AP2112K-3.3
- removed U3: 74HCT244, Package_SO:SOIC-20W_7.5x12.8mm_P1.27mm, symbol 74xx:74HCT244
- removed U4: SN65HVD230, Package_SO:SOIC-8_3.9x4.9mm_P1.27mm, symbol Interface_CAN_LIN:SN65HVD230
- removed U5: PC817, Package_DIP:DIP-4_W7.62mm, symbol Isolator:PC817
Connections:
- no-connect marks 9 -> 0
Other:
- added sheet 12 V input and protection (input.kicad_sch)
- added sheet 3.3 V, the pod's 5 V, the LiDAR feed (rails.kicad_sch)
- added sheet 5 V converter (TPS54360, TI reference design) (buck.kicad_sch)
- added sheet Brake actuator: buffer, BTS7960, current sense, cable magnet (actuator.kicad_sch)
- added sheet CAN transceiver for OBD-II (can.kicad_sch)
- added sheet Inter-box cable: DB-25 to the pod (cable.kicad_sch)
- added sheet Presence, brake light, E-stop sense, kill relay, bench (status.kicad_sch)
- added sheet Signal relays: indicators, hazards, horn, high beam (relays.kicad_sch)
- note added: "12 V input -> 5 V converter -> 3.3 V and the pod's 5 V. The pod drives the actuator, relays and CAN; the status sheet reports back to it."
- note added: "UNDER-DASH POWER BOARD: block diagram. Each box is a sheet (double-click it in KiCad). Power rails +12V, +5V, +3V3 and GND join the sheets by name (power symbols); every other connection between sheets is a wire here."
- note removed: "12 V input: fuse, TVS, reverse-polarity diode"
- note removed: "3.3 V, pod supply, LiDAR feed"
- note removed: "5 V: TPS54360 (TI reference design, 600 kHz)"
- note removed: "Brake actuator: buffer, BTS7960, current sense, cable magnet"
- note removed: "CAN transceiver, presence, brake light, E-stop, bench"
- note removed: "Fail-safe pull-downs (Part 4.8.4)"
- note removed: "Inter-box cable (DB-25), BUILD_GUIDE 4.8.3"
- note removed: "Mounting"
- note removed: "Signal relays (active-high, low-side MOSFETs)"

Commit message: PCBs routed, labelled and ready to order: Rev 1 fabrication files and buy list
Both boards placed, routed and finished by script (hardware/gen): layout.sh places
(placement.py, with silkscreen names for every terminal, port, header and button),
route.sh routes with Freerouting inside rule areas and net classes from the layout
guide and keeps a board only with 0 DRC errors, 0 unconnected and exact schematic
parity, routespec.sh checks what the DRC cannot (planes, crystal, converter loop,
IPC-2221 widths), finish.sh adds the bottom-silkscreen identification and writes
the fabrication files (gerbers, drill, BOM, positions) only when the DRC passes.

- Pod 70 x 53 mm, 4 layers: In1 solid GND, In2 +3V3, 530 teardrops; no DRC warnings.
- Power 95 x 66 mm, 2 layers, 2 oz: 10 A rail as a zone, converter re-placed (switch
  node 16 mm, feedback 7 mm, no vias; was 78 mm and 40 mm), 328 teardrops.
- Screw terminals turned to open outward; RESET/BOOT side-push on the pod's left
  edge; USB-C footprint with a 3D model (GCT USB4105).
- Pod J2 now the Adafruit 4754's JP1 row pin for pin (the old order shorted its
  3.3 V output to ground); IMU reset on a new J8; HC-05 header fed 5 V.
- Buy list per footprint and module connections in bill-of-materials.md section 10.
- LAYOUT_GUIDE rewritten as how the boards were routed and how to review them;
  decisions, progress log and BUILD_GUIDE updated; power box follows the wider board.
Changed lines of the file:
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@@
 		(instances
 			(project "power_board"
-				(path "/244ac675-494c-4e27-8819-02215b480bc3"
+				(path "/c794bf93-11d2-4d5c-a02b-6bb49c306097"
 					(page "9")
 				)
@@
 		(instances
 			(project "power_board"
-				(path "/244ac675-494c-4e27-8819-02215b480bc3"
+				(path "/c794bf93-11d2-4d5c-a02b-6bb49c306097"
 					(page "4")
 				)
@@
 		(instances
 			(project "power_board"
-				(path "/244ac675-494c-4e27-8819-02215b480bc3"
+				(path "/c794bf93-11d2-4d5c-a02b-6bb49c306097"
 					(page "5")
 				)
@@
 		(instances
 			(project "power_board"
-				(path "/244ac675-494c-4e27-8819-02215b480bc3"
+				(path "/c794bf93-11d2-4d5c-a02b-6bb49c306097"
 					(page "6")
 				)
@@
 		(instances
 			(project "power_board"
-				(path "/244ac675-494c-4e27-8819-02215b480bc3"
+				(path "/c794bf93-11d2-4d5c-a02b-6bb49c306097"
 					(page "7")
 				)
@@
 		(instances
 			(project "power_board"
-				(path "/244ac675-494c-4e27-8819-02215b480bc3"
+				(path "/c794bf93-11d2-4d5c-a02b-6bb49c306097"
 					(page "8")
 				)
@@
 		(instances
 			(project "power_board"
-				(path "/244ac675-494c-4e27-8819-02215b480bc3"
+				(path "/c794bf93-11d2-4d5c-a02b-6bb49c306097"
 					(page "2")
 				)
@@
 		(instances
 			(project "power_board"
-				(path "/244ac675-494c-4e27-8819-02215b480bc3"
+				(path "/c794bf93-11d2-4d5c-a02b-6bb49c306097"
 					(page "3")
 				)
@@
 	(wire
 		(pts
-			(xy 193.04 59.69)
-			(xy 118.11 59.69)
-		)
-		(stroke
-			(width 0)
-			(type default)
-		)
-	)
-	(wire
-		(pts
 			(xy 116.84 59.69)
 			(xy 118.11 59.69)
@@
 	(wire
 		(pts
-			(xy 193.04 140.97)
-			(xy 118.11 140.97)
+			(xy 118.11 59.69)
+			(xy 193.04 59.69)
 		)
 		(stroke
@@
 	(wire
 		(pts
-			(xy 193.04 80.01)
-			(xy 118.11 80.01)
+			(xy 118.11 140.97)
+			(xy 193.04 140.97)
 		)
 		(stroke
@@
 	(wire
 		(pts
+			(xy 118.11 80.01)
+			(xy 193.04 80.01)
+		)
+		(stroke
+			(width 0)
+			(type default)
+		)
+	)
+	(wire
+		(pts
+			(xy 116.84 74.93)
+			(xy 118.11 74.93)
+		)
+		(stroke
+			(width 0)
+			(type default)
+		)
+	)
+	(wire
+		(pts
 			(xy 118.11 74.93)
 			(xy 193.04 74.93)
@@
 	(wire
 		(pts
-			(xy 116.84 74.93)
-			(xy 118.11 74.93)
-		)
-		(stroke
-			(width 0)
-			(type default)
-		)
-	)
-	(wire
-		(pts
+			(xy 116.84 143.51)
 			(xy 118.11 143.51)
-			(xy 116.84 143.51)
 		)
 		(stroke
@@
 	(wire
 		(pts
+			(xy 116.84 72.39)
+			(xy 118.11 72.39)
+		)
+		(stroke
+			(width 0)
+			(type default)
+		)
+	)
+	(wire
+		(pts
+			(xy 118.11 72.39)
 			(xy 193.04 72.39)
-			(xy 118.11 72.39)
-		)
-		(stroke
-			(width 0)
-			(type default)
-		)
-	)
-	(wire
-		(pts
-			(xy 118.11 72.39)
-			(xy 116.84 72.39)
+		)
+		(stroke
+			(width 0)
+			(type default)
+		)
+	)
+	(wire
+		(pts
+			(xy 116.84 69.85)
+			(xy 118.11 69.85)
 		)
 		(stroke
@@
 	(wire
 		(pts
-			(xy 116.84 69.85)
-			(xy 118.11 69.85)
-		)
-		(stroke
-			(width 0)
-			(type default)
-		)
-	)
-	(wire
-		(pts
-			(xy 193.04 123.19)
-			(xy 118.11 123.19)
-		)
-		(stroke
-			(width 0)
-			(type default)
-		)
-	)
-	(wire
-		(pts
 			(xy 116.84 123.19)
 			(xy 118.11 123.19)
@@
 	(wire
 		(pts
+			(xy 118.11 123.19)
+			(xy 193.04 123.19)
+		)
+		(stroke
+			(width 0)
+			(type default)
+		)
+	)
+	(wire
+		(pts
+			(xy 116.84 125.73)
+			(xy 118.11 125.73)
+		)
+		(stroke
+			(width 0)
+			(type default)
+		)
+	)
+	(wire
+		(pts
 			(xy 118.11 125.73)
 			(xy 193.04 125.73)
@@
 	(wire
 		(pts
-			(xy 116.84 125.73)
-			(xy 118.11 125.73)
+			(xy 116.84 120.65)
+			(xy 118.11 120.65)
 		)
 		(stroke
@@
 	(wire
 		(pts
-			(xy 116.84 120.65)
-			(xy 118.11 120.65)
-		)
-		(stroke
-			(width 0)
-			(type default)
-		)
-	)
-	(wire
-		(pts
-			(xy 193.04 148.59)
-			(xy 118.11 148.59)
-		)
-		(stroke
-			(width 0)
-			(type default)
-		)
-	)
-	(wire
-		(pts
 			(xy 116.84 148.59)
 			(xy 118.11 148.59)
@@
 	(wire
 		(pts
+			(xy 118.11 148.59)
+			(xy 193.04 148.59)
+		)
+		(stroke
+			(width 0)
+			(type default)
+		)
+	)
+	(wire
+		(pts
+			(xy 116.84 151.13)
+			(xy 118.11 151.13)
+		)
+		(stroke
+			(width 0)
+			(type default)
+		)
+	)
+	(wire
+		(pts
 			(xy 118.11 151.13)
 			(xy 193.04 151.13)
@@
 	(wire
 		(pts
-			(xy 118.11 151.13)
-			(xy 116.84 151.13)
-		)
-		(stroke
-			(width 0)
-			(type default)
-		)
-	)
-	(wire
-		(pts
-			(xy 193.04 146.05)
-			(xy 118.11 146.05)
-		)
-		(stroke
-			(width 0)
-			(type default)
-		)
-	)
-	(wire
-		(pts
 			(xy 116.84 146.05)
 			(xy 118.11 146.05)
@@
 	(wire
 		(pts
+			(xy 118.11 146.05)
+			(xy 193.04 146.05)
+		)
+		(stroke
+			(width 0)
+			(type default)
+		)
+	)
+	(wire
+		(pts
+			(xy 116.84 77.47)
+			(xy 118.11 77.47)
+		)
+		(stroke
+			(width 0)
+			(type default)
+		)
+	)
+	(wire
+		(pts
 			(xy 118.11 77.47)
 			(xy 193.04 77.47)
@@
 	(wire
 		(pts
-			(xy 116.84 77.47)
-			(xy 118.11 77.47)
+			(xy 116.84 105.41)
+			(xy 118.11 105.41)
 		)
 		(stroke
@@
 	(wire
 		(pts
-			(xy 116.84 105.41)
-			(xy 118.11 105.41)
+			(xy 116.84 100.33)
+			(xy 118.11 100.33)
 		)
 		(stroke
@@
 	(wire
 		(pts
-			(xy 118.11 100.33)
-			(xy 116.84 100.33)
-		)
-		(stroke
-			(width 0)
-			(type default)
-		)
-	)
-	(wire
-		(pts
-			(xy 193.04 102.87)
-			(xy 118.11 102.87)
-		)
-		(stroke
-			(width 0)
-			(type default)
-		)
-	)
-	(wire
-		(pts
 			(xy 116.84 102.87)
 			(xy 118.11 102.87)
@@
 	(wire
 		(pts
-			(xy 193.04 95.25)
-			(xy 118.11 95.25)
+			(xy 118.11 102.87)
+			(xy 193.04 102.87)
 		)
 		(stroke
@@
 	(wire
 		(pts
+			(xy 118.11 95.25)
+			(xy 193.04 95.25)
+		)
+		(stroke
+			(width 0)
+			(type default)
+		)
+	)
+	(wire
+		(pts
+			(xy 116.84 97.79)
+			(xy 118.11 97.79)
+		)
+		(stroke
+			(width 0)
+			(type default)
+		)
+	)
+	(wire
+		(pts
 			(xy 118.11 97.79)
 			(xy 193.04 97.79)
 		)
 		(stroke
-			(width 0)
-			(type default)
-		)
-	)
-	(wire
-		(pts
-			(xy 116.84 97.79)
-			(xy 118.11 97.79)
-		)
-		(stroke
