File: hardware/power_board/rails.kicad_sch (KiCad schematic)
At the start: 7 parts, among them J3 LiDAR 12 V out, U2 AP2112K-3.3

Commit message: Pod board schematic redrawn as wired sheets; duplicate references fixed
pod_board_drawing.py draws six sheets around an MCU sheet under a block
diagram; check.sh now compares both boards' drawn and label-only netlists.
kisheet.py: stacked pins, PWR_FLAGs on signal nets, column hints for
crossing-free fan-ins, nets drawn in pieces joined by name, and visible
rail names on power symbols.

R31-R33 were used twice on the pod board, which KiCad's ERC does not
report; the netlist merged each pair. Cable parts now start at R40/C40,
generate.py rejects duplicate references and check_nets.py fails on a pin
in two nets. check_nets.py also drops the sheet path from net names.
Changed lines of the file:
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@@
 		(instances
 			(project "power_board"
-				(path "/3aef661e-32a5-4098-b535-e9581569514f/039a3234-7946-4146-b26f-7d4ce0570526"
+				(path "/244ac675-494c-4e27-8819-02215b480bc3/1c999e15-334d-4028-92b9-7bb391690306"
 					(reference "U2")
 					(unit 1)
@@
 		(instances
 			(project "power_board"
-				(path "/3aef661e-32a5-4098-b535-e9581569514f/039a3234-7946-4146-b26f-7d4ce0570526"
+				(path "/244ac675-494c-4e27-8819-02215b480bc3/1c999e15-334d-4028-92b9-7bb391690306"
 					(reference "C28")
 					(unit 1)
@@
 		(instances
 			(project "power_board"
-				(path "/3aef661e-32a5-4098-b535-e9581569514f/039a3234-7946-4146-b26f-7d4ce0570526"
+				(path "/244ac675-494c-4e27-8819-02215b480bc3/1c999e15-334d-4028-92b9-7bb391690306"
 					(reference "C29")
 					(unit 1)
@@
 		(instances
 			(project "power_board"
-				(path "/3aef661e-32a5-4098-b535-e9581569514f/039a3234-7946-4146-b26f-7d4ce0570526"
+				(path "/244ac675-494c-4e27-8819-02215b480bc3/1c999e15-334d-4028-92b9-7bb391690306"
 					(reference "F2")
 					(unit 1)
@@
 		(instances
 			(project "power_board"
-				(path "/3aef661e-32a5-4098-b535-e9581569514f/039a3234-7946-4146-b26f-7d4ce0570526"
+				(path "/244ac675-494c-4e27-8819-02215b480bc3/1c999e15-334d-4028-92b9-7bb391690306"
 					(reference "C30")
 					(unit 1)
@@
 		(instances
 			(project "power_board"
-				(path "/3aef661e-32a5-4098-b535-e9581569514f/039a3234-7946-4146-b26f-7d4ce0570526"
+				(path "/244ac675-494c-4e27-8819-02215b480bc3/1c999e15-334d-4028-92b9-7bb391690306"
 					(reference "F3")
 					(unit 1)
@@
 		(instances
 			(project "power_board"
-				(path "/3aef661e-32a5-4098-b535-e9581569514f/039a3234-7946-4146-b26f-7d4ce0570526"
+				(path "/244ac675-494c-4e27-8819-02215b480bc3/1c999e15-334d-4028-92b9-7bb391690306"
 					(reference "J3")
 					(unit 1)
@@
 		)
 		(property "Value" "+5V"
-			(at 60.96 63.5 0)
-			(hide yes)
-			(effects
-				(font
-					(size 1.0 1.0)
+			(at 60.96 59.9 0)
+			(effects
+				(font
+					(size 1.27 1.27)
 				)
 			)
@@
 		(instances
 			(project "power_board"
-				(path "/3aef661e-32a5-4098-b535-e9581569514f/039a3234-7946-4146-b26f-7d4ce0570526"
+				(path "/244ac675-494c-4e27-8819-02215b480bc3/1c999e15-334d-4028-92b9-7bb391690306"
 					(reference "#PWR023")
 					(unit 1)
@@
 		)
 		(property "Value" "+3V3"
-			(at 137.16 63.5 0)
-			(hide yes)
-			(effects
-				(font
-					(size 1.0 1.0)
+			(at 137.16 59.9 0)
+			(effects
+				(font
+					(size 1.27 1.27)
 				)
 			)
@@
 		(instances
 			(project "power_board"
-				(path "/3aef661e-32a5-4098-b535-e9581569514f/039a3234-7946-4146-b26f-7d4ce0570526"
+				(path "/244ac675-494c-4e27-8819-02215b480bc3/1c999e15-334d-4028-92b9-7bb391690306"
 					(reference "#PWR024")
 					(unit 1)
@@
 		)
 		(property "Value" "GND"
-			(at 101.6 86.36 0)
-			(hide yes)
-			(effects
-				(font
-					(size 1.0 1.0)
+			(at 101.6 82.76 0)
+			(hide yes)
+			(effects
+				(font
+					(size 1.27 1.27)
 				)
 			)
@@
 		(instances
 			(project "power_board"
-				(path "/3aef661e-32a5-4098-b535-e9581569514f/039a3234-7946-4146-b26f-7d4ce0570526"
+				(path "/244ac675-494c-4e27-8819-02215b480bc3/1c999e15-334d-4028-92b9-7bb391690306"
 					(reference "#PWR025")
 					(unit 1)
@@
 		)
 		(property "Value" "GND"
-			(at 76.2 87.63 0)
-			(hide yes)
-			(effects
-				(font
-					(size 1.0 1.0)
+			(at 76.2 84.03 0)
+			(hide yes)
+			(effects
+				(font
+					(size 1.27 1.27)
 				)
 			)
@@
 		(instances
 			(project "power_board"
-				(path "/3aef661e-32a5-4098-b535-e9581569514f/039a3234-7946-4146-b26f-7d4ce0570526"
+				(path "/244ac675-494c-4e27-8819-02215b480bc3/1c999e15-334d-4028-92b9-7bb391690306"
 					(reference "#PWR026")
 					(unit 1)
@@
 		)
 		(property "Value" "GND"
-			(at 121.92 87.63 0)
-			(hide yes)
-			(effects
-				(font
-					(size 1.0 1.0)
+			(at 121.92 84.03 0)
+			(hide yes)
+			(effects
+				(font
+					(size 1.27 1.27)
 				)
 			)
@@
 		(instances
 			(project "power_board"
-				(path "/3aef661e-32a5-4098-b535-e9581569514f/039a3234-7946-4146-b26f-7d4ce0570526"
+				(path "/244ac675-494c-4e27-8819-02215b480bc3/1c999e15-334d-4028-92b9-7bb391690306"
 					(reference "#PWR027")
 					(unit 1)
@@
 		)
 		(property "Value" "+5V"
-			(at 85.09 119.38 0)
-			(hide yes)
-			(effects
-				(font
-					(size 1.0 1.0)
+			(at 85.09 115.78 0)
+			(effects
+				(font
+					(size 1.27 1.27)
 				)
 			)
@@
 		(instances
 			(project "power_board"
-				(path "/3aef661e-32a5-4098-b535-e9581569514f/039a3234-7946-4146-b26f-7d4ce0570526"
+				(path "/244ac675-494c-4e27-8819-02215b480bc3/1c999e15-334d-4028-92b9-7bb391690306"
 					(reference "#PWR028")
 					(unit 1)
@@
 		)
 		(property "Value" "GND"
-			(at 111.76 135.89 0)
-			(hide yes)
-			(effects
-				(font
-					(size 1.0 1.0)
+			(at 111.76 132.29 0)
+			(hide yes)
+			(effects
+				(font
+					(size 1.27 1.27)
 				)
 			)
@@
 		(instances
 			(project "power_board"
-				(path "/3aef661e-32a5-4098-b535-e9581569514f/039a3234-7946-4146-b26f-7d4ce0570526"
+				(path "/244ac675-494c-4e27-8819-02215b480bc3/1c999e15-334d-4028-92b9-7bb391690306"
 					(reference "#PWR029")
 					(unit 1)
@@
 		)
 		(property "Value" "+12V"
-			(at 85.09 160.02 0)
-			(hide yes)
-			(effects
-				(font
-					(size 1.0 1.0)
+			(at 85.09 156.42 0)
+			(effects
+				(font
+					(size 1.27 1.27)
 				)
 			)
@@
 		(instances
 			(project "power_board"
-				(path "/3aef661e-32a5-4098-b535-e9581569514f/039a3234-7946-4146-b26f-7d4ce0570526"
+				(path "/244ac675-494c-4e27-8819-02215b480bc3/1c999e15-334d-4028-92b9-7bb391690306"
 					(reference "#PWR030")
 					(unit 1)
@@
 		)
 		(property "Value" "GND"
-			(at 124.46 167.64 0)
-			(hide yes)
-			(effects
-				(font
-					(size 1.0 1.0)
+			(at 124.46 164.04 0)
+			(hide yes)
+			(effects
+				(font
+					(size 1.27 1.27)
 				)
 			)
@@
 		(instances
 			(project "power_board"
-				(path "/3aef661e-32a5-4098-b535-e9581569514f/039a3234-7946-4146-b26f-7d4ce0570526"
+				(path "/244ac675-494c-4e27-8819-02215b480bc3/1c999e15-334d-4028-92b9-7bb391690306"
 					(reference "#PWR031")
 					(unit 1)

Commit message: PCBs routed, labelled and ready to order: Rev 1 fabrication files and buy list
Both boards placed, routed and finished by script (hardware/gen): layout.sh places
(placement.py, with silkscreen names for every terminal, port, header and button),
route.sh routes with Freerouting inside rule areas and net classes from the layout
guide and keeps a board only with 0 DRC errors, 0 unconnected and exact schematic
parity, routespec.sh checks what the DRC cannot (planes, crystal, converter loop,
IPC-2221 widths), finish.sh adds the bottom-silkscreen identification and writes
the fabrication files (gerbers, drill, BOM, positions) only when the DRC passes.

- Pod 70 x 53 mm, 4 layers: In1 solid GND, In2 +3V3, 530 teardrops; no DRC warnings.
- Power 95 x 66 mm, 2 layers, 2 oz: 10 A rail as a zone, converter re-placed (switch
  node 16 mm, feedback 7 mm, no vias; was 78 mm and 40 mm), 328 teardrops.
- Screw terminals turned to open outward; RESET/BOOT side-push on the pod's left
  edge; USB-C footprint with a 3D model (GCT USB4105).
- Pod J2 now the Adafruit 4754's JP1 row pin for pin (the old order shorted its
  3.3 V output to ground); IMU reset on a new J8; HC-05 header fed 5 V.
- Buy list per footprint and module connections in bill-of-materials.md section 10.
- LAYOUT_GUIDE rewritten as how the boards were routed and how to review them;
  decisions, progress log and BUILD_GUIDE updated; power box follows the wider board.
Changed lines of the file:
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@@
 		(instances
 			(project "power_board"
-				(path "/244ac675-494c-4e27-8819-02215b480bc3/1c999e15-334d-4028-92b9-7bb391690306"
+				(path "/c794bf93-11d2-4d5c-a02b-6bb49c306097/d133e5b5-c332-4484-b87b-0d8ef32544df"
 					(reference "U2")
 					(unit 1)
@@
 		(instances
 			(project "power_board"
-				(path "/244ac675-494c-4e27-8819-02215b480bc3/1c999e15-334d-4028-92b9-7bb391690306"
+				(path "/c794bf93-11d2-4d5c-a02b-6bb49c306097/d133e5b5-c332-4484-b87b-0d8ef32544df"
 					(reference "C28")
 					(unit 1)
@@
 		(instances
 			(project "power_board"
-				(path "/244ac675-494c-4e27-8819-02215b480bc3/1c999e15-334d-4028-92b9-7bb391690306"
+				(path "/c794bf93-11d2-4d5c-a02b-6bb49c306097/d133e5b5-c332-4484-b87b-0d8ef32544df"
 					(reference "C29")
 					(unit 1)
@@
 		(instances
 			(project "power_board"
-				(path "/244ac675-494c-4e27-8819-02215b480bc3/1c999e15-334d-4028-92b9-7bb391690306"
+				(path "/c794bf93-11d2-4d5c-a02b-6bb49c306097/d133e5b5-c332-4484-b87b-0d8ef32544df"
 					(reference "F2")
 					(unit 1)
@@
 		(instances
 			(project "power_board"
-				(path "/244ac675-494c-4e27-8819-02215b480bc3/1c999e15-334d-4028-92b9-7bb391690306"
+				(path "/c794bf93-11d2-4d5c-a02b-6bb49c306097/d133e5b5-c332-4484-b87b-0d8ef32544df"
 					(reference "C30")
 					(unit 1)
@@
 		(instances
 			(project "power_board"
-				(path "/244ac675-494c-4e27-8819-02215b480bc3/1c999e15-334d-4028-92b9-7bb391690306"
+				(path "/c794bf93-11d2-4d5c-a02b-6bb49c306097/d133e5b5-c332-4484-b87b-0d8ef32544df"
 					(reference "F3")
 					(unit 1)
@@
 		(instances
 			(project "power_board"
-				(path "/244ac675-494c-4e27-8819-02215b480bc3/1c999e15-334d-4028-92b9-7bb391690306"
+				(path "/c794bf93-11d2-4d5c-a02b-6bb49c306097/d133e5b5-c332-4484-b87b-0d8ef32544df"
 					(reference "J3")
 					(unit 1)
@@
 		(instances
 			(project "power_board"
-				(path "/244ac675-494c-4e27-8819-02215b480bc3/1c999e15-334d-4028-92b9-7bb391690306"
+				(path "/c794bf93-11d2-4d5c-a02b-6bb49c306097/d133e5b5-c332-4484-b87b-0d8ef32544df"
 					(reference "#PWR023")
 					(unit 1)
@@
 		(instances
 			(project "power_board"
-				(path "/244ac675-494c-4e27-8819-02215b480bc3/1c999e15-334d-4028-92b9-7bb391690306"
+				(path "/c794bf93-11d2-4d5c-a02b-6bb49c306097/d133e5b5-c332-4484-b87b-0d8ef32544df"
 					(reference "#PWR024")
 					(unit 1)
@@
 		(instances
 			(project "power_board"
-				(path "/244ac675-494c-4e27-8819-02215b480bc3/1c999e15-334d-4028-92b9-7bb391690306"
+				(path "/c794bf93-11d2-4d5c-a02b-6bb49c306097/d133e5b5-c332-4484-b87b-0d8ef32544df"
 					(reference "#PWR025")
 					(unit 1)
@@
 		(instances
 			(project "power_board"
-				(path "/244ac675-494c-4e27-8819-02215b480bc3/1c999e15-334d-4028-92b9-7bb391690306"
+				(path "/c794bf93-11d2-4d5c-a02b-6bb49c306097/d133e5b5-c332-4484-b87b-0d8ef32544df"
 					(reference "#PWR026")
 					(unit 1)
@@
 		(instances
 			(project "power_board"
-				(path "/244ac675-494c-4e27-8819-02215b480bc3/1c999e15-334d-4028-92b9-7bb391690306"
+				(path "/c794bf93-11d2-4d5c-a02b-6bb49c306097/d133e5b5-c332-4484-b87b-0d8ef32544df"
 					(reference "#PWR027")
 					(unit 1)
@@
 		(instances
 			(project "power_board"
-				(path "/244ac675-494c-4e27-8819-02215b480bc3/1c999e15-334d-4028-92b9-7bb391690306"
+				(path "/c794bf93-11d2-4d5c-a02b-6bb49c306097/d133e5b5-c332-4484-b87b-0d8ef32544df"
 					(reference "#PWR028")
 					(unit 1)
@@
 		(instances
 			(project "power_board"
-				(path "/244ac675-494c-4e27-8819-02215b480bc3/1c999e15-334d-4028-92b9-7bb391690306"
+				(path "/c794bf93-11d2-4d5c-a02b-6bb49c306097/d133e5b5-c332-4484-b87b-0d8ef32544df"
 					(reference "#PWR029")
 					(unit 1)
@@
 		(instances
 			(project "power_board"
-				(path "/244ac675-494c-4e27-8819-02215b480bc3/1c999e15-334d-4028-92b9-7bb391690306"
+				(path "/c794bf93-11d2-4d5c-a02b-6bb49c306097/d133e5b5-c332-4484-b87b-0d8ef32544df"
 					(reference "#PWR030")
 					(unit 1)
@@
 		(instances
 			(project "power_board"
-				(path "/244ac675-494c-4e27-8819-02215b480bc3/1c999e15-334d-4028-92b9-7bb391690306"
+				(path "/c794bf93-11d2-4d5c-a02b-6bb49c306097/d133e5b5-c332-4484-b87b-0d8ef32544df"
 					(reference "#PWR031")
 					(unit 1)
@@
 	(wire
 		(pts
+			(xy 95.25 162.56)
+			(xy 96.52 162.56)
+		)
+		(stroke
+			(width 0)
+			(type default)
+		)
+	)
+	(wire
+		(pts
 			(xy 96.52 162.56)
 			(xy 127.0 162.56)
@@
 	(wire
 		(pts
-			(xy 95.25 162.56)
-			(xy 96.52 162.56)
-		)
-		(stroke
-			(width 0)
-			(type default)
-		)
-	)
-	(wire
-		(pts
+			(xy 109.22 73.66)
 			(xy 121.92 73.66)
-			(xy 109.22 73.66)
 		)
 		(stroke
@@
 	(wire
 		(pts
+			(xy 60.96 63.5)
+			(xy 60.96 64.77)
+		)
+		(stroke
+			(width 0)
+			(type default)
+		)
+	)
+	(wire
+		(pts
+			(xy 60.96 64.77)
+			(xy 76.2 64.77)
+		)
+		(stroke
+			(width 0)
+			(type default)
+		)
+	)
+	(wire
+		(pts
+			(xy 76.2 64.77)
+			(xy 76.2 73.66)
+		)
+		(stroke
+			(width 0)
+			(type default)
+		)
+	)
+	(wire
+		(pts
+			(xy 76.2 73.66)
+			(xy 76.2 77.47)
+		)
+		(stroke
+			(width 0)
+			(type default)
+		)
+	)
+	(wire
+		(pts
 			(xy 76.2 73.66)
 			(xy 92.71 73.66)
@@
 	(wire
 		(pts
-			(xy 60.96 64.77)
-			(xy 76.2 64.77)
-		)
-		(stroke
-			(width 0)
-			(type default)
-		)
-	)
-	(wire
-		(pts
-			(xy 76.2 73.66)
-			(xy 76.2 64.77)
+			(xy 92.71 73.66)
+			(xy 92.71 76.2)
+		)
+		(stroke
+			(width 0)
+			(type default)
+		)
+	)
+	(wire
+		(pts
+			(xy 92.71 73.66)
+			(xy 93.98 73.66)
 		)
 		(stroke
@@
 			(xy 92.71 76.2)
 			(xy 93.98 76.2)
-		)
-		(stroke
-			(width 0)
-			(type default)
-		)
-	)
-	(wire
-		(pts
-			(xy 92.71 73.66)
-			(xy 93.98 73.66)
-		)
-		(stroke
-			(width 0)
-			(type default)
-		)
-	)
-	(wire
-		(pts
-			(xy 76.2 73.66)
-			(xy 76.2 77.47)
-		)
-		(stroke
-			(width 0)
-			(type default)
-		)
-	)
-	(wire
-		(pts
-			(xy 92.71 73.66)
-			(xy 92.71 76.2)
-		)
-		(stroke
-			(width 0)
-			(type default)
-		)
-	)
-	(wire
-		(pts
-			(xy 60.96 63.5)
-			(xy 60.96 64.77)
 		)
 		(stroke
@@
 	(wire
 		(pts
-			(xy 266.7 121.92)
-			(xy 111.76 121.92)
-		)
-		(stroke
-			(width 0)
-			(type default)
-		)
-	)
-	(wire
-		(pts
 			(xy 95.25 121.92)
 			(xy 111.76 121.92)
@@
 		)
 		(stroke
+			(width 0)
+			(type default)
+		)
+	)
+	(wire
+		(pts
+			(xy 111.76 121.92)
+			(xy 266.7 121.92)
+		)
+		(stroke
