File: hardware/power_board/status.kicad_sch (KiCad schematic)
At the start: 10 parts, among them J10 Brake-light switch, J12 Bench: HX711, J8 Kill relay coil feed, J9 E-stop sense contact, Q8 2N7002, U5 PC817

Commit message: Pod board schematic redrawn as wired sheets; duplicate references fixed
pod_board_drawing.py draws six sheets around an MCU sheet under a block
diagram; check.sh now compares both boards' drawn and label-only netlists.
kisheet.py: stacked pins, PWR_FLAGs on signal nets, column hints for
crossing-free fan-ins, nets drawn in pieces joined by name, and visible
rail names on power symbols.

R31-R33 were used twice on the pod board, which KiCad's ERC does not
report; the netlist merged each pair. Cable parts now start at R40/C40,
generate.py rejects duplicate references and check_nets.py fails on a pin
in two nets. check_nets.py also drops the sheet path from net names.
Changed lines of the file:
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@@
 		(instances
 			(project "power_board"
-				(path "/3aef661e-32a5-4098-b535-e9581569514f/20733ad5-b1e0-4da3-932e-70bddfad2269"
+				(path "/244ac675-494c-4e27-8819-02215b480bc3/2561dbd3-5769-4d66-b028-2cb47955e72c"
 					(reference "Q8")
 					(unit 1)
@@
 		(instances
 			(project "power_board"
-				(path "/3aef661e-32a5-4098-b535-e9581569514f/20733ad5-b1e0-4da3-932e-70bddfad2269"
+				(path "/244ac675-494c-4e27-8819-02215b480bc3/2561dbd3-5769-4d66-b028-2cb47955e72c"
 					(reference "R61")
 					(unit 1)
@@
 		(instances
 			(project "power_board"
-				(path "/3aef661e-32a5-4098-b535-e9581569514f/20733ad5-b1e0-4da3-932e-70bddfad2269"
+				(path "/244ac675-494c-4e27-8819-02215b480bc3/2561dbd3-5769-4d66-b028-2cb47955e72c"
 					(reference "R62")
 					(unit 1)
@@
 		(instances
 			(project "power_board"
-				(path "/3aef661e-32a5-4098-b535-e9581569514f/20733ad5-b1e0-4da3-932e-70bddfad2269"
+				(path "/244ac675-494c-4e27-8819-02215b480bc3/2561dbd3-5769-4d66-b028-2cb47955e72c"
 					(reference "J10")
 					(unit 1)
@@
 		(instances
 			(project "power_board"
-				(path "/3aef661e-32a5-4098-b535-e9581569514f/20733ad5-b1e0-4da3-932e-70bddfad2269"
+				(path "/244ac675-494c-4e27-8819-02215b480bc3/2561dbd3-5769-4d66-b028-2cb47955e72c"
 					(reference "R63")
 					(unit 1)
@@
 		(instances
 			(project "power_board"
-				(path "/3aef661e-32a5-4098-b535-e9581569514f/20733ad5-b1e0-4da3-932e-70bddfad2269"
+				(path "/244ac675-494c-4e27-8819-02215b480bc3/2561dbd3-5769-4d66-b028-2cb47955e72c"
 					(reference "U5")
 					(unit 1)
@@
 		(instances
 			(project "power_board"
-				(path "/3aef661e-32a5-4098-b535-e9581569514f/20733ad5-b1e0-4da3-932e-70bddfad2269"
+				(path "/244ac675-494c-4e27-8819-02215b480bc3/2561dbd3-5769-4d66-b028-2cb47955e72c"
 					(reference "D21")
 					(unit 1)
@@
 		(instances
 			(project "power_board"
-				(path "/3aef661e-32a5-4098-b535-e9581569514f/20733ad5-b1e0-4da3-932e-70bddfad2269"
+				(path "/244ac675-494c-4e27-8819-02215b480bc3/2561dbd3-5769-4d66-b028-2cb47955e72c"
 					(reference "J9")
 					(unit 1)
@@
 		(instances
 			(project "power_board"
-				(path "/3aef661e-32a5-4098-b535-e9581569514f/20733ad5-b1e0-4da3-932e-70bddfad2269"
+				(path "/244ac675-494c-4e27-8819-02215b480bc3/2561dbd3-5769-4d66-b028-2cb47955e72c"
 					(reference "J8")
 					(unit 1)
@@
 		(instances
 			(project "power_board"
-				(path "/3aef661e-32a5-4098-b535-e9581569514f/20733ad5-b1e0-4da3-932e-70bddfad2269"
+				(path "/244ac675-494c-4e27-8819-02215b480bc3/2561dbd3-5769-4d66-b028-2cb47955e72c"
 					(reference "J12")
 					(unit 1)
@@
 		)
 		(property "Value" "GND"
-			(at 99.06 68.58 0)
-			(hide yes)
-			(effects
-				(font
-					(size 1.0 1.0)
+			(at 99.06 64.98 0)
+			(hide yes)
+			(effects
+				(font
+					(size 1.27 1.27)
 				)
 			)
@@
 		(instances
 			(project "power_board"
-				(path "/3aef661e-32a5-4098-b535-e9581569514f/20733ad5-b1e0-4da3-932e-70bddfad2269"
+				(path "/244ac675-494c-4e27-8819-02215b480bc3/2561dbd3-5769-4d66-b028-2cb47955e72c"
 					(reference "#PWR072")
 					(unit 1)
@@
 		)
 		(property "Value" "+5V"
-			(at 121.92 46.99 0)
-			(hide yes)
-			(effects
-				(font
-					(size 1.0 1.0)
+			(at 121.92 43.39 0)
+			(effects
+				(font
+					(size 1.27 1.27)
 				)
 			)
@@
 		(instances
 			(project "power_board"
-				(path "/3aef661e-32a5-4098-b535-e9581569514f/20733ad5-b1e0-4da3-932e-70bddfad2269"
+				(path "/244ac675-494c-4e27-8819-02215b480bc3/2561dbd3-5769-4d66-b028-2cb47955e72c"
 					(reference "#PWR073")
 					(unit 1)
@@
 		)
 		(property "Value" "GND"
-			(at 121.92 80.01 0)
-			(hide yes)
-			(effects
-				(font
-					(size 1.0 1.0)
+			(at 121.92 76.41 0)
+			(hide yes)
+			(effects
+				(font
+					(size 1.27 1.27)
 				)
 			)
@@
 		(instances
 			(project "power_board"
-				(path "/3aef661e-32a5-4098-b535-e9581569514f/20733ad5-b1e0-4da3-932e-70bddfad2269"
+				(path "/244ac675-494c-4e27-8819-02215b480bc3/2561dbd3-5769-4d66-b028-2cb47955e72c"
 					(reference "#PWR074")
 					(unit 1)
@@
 		)
 		(property "Value" "GND"
-			(at 256.54 106.68 0)
-			(hide yes)
-			(effects
-				(font
-					(size 1.0 1.0)
+			(at 256.54 103.08 0)
+			(hide yes)
+			(effects
+				(font
+					(size 1.27 1.27)
 				)
 			)
@@
 		(instances
 			(project "power_board"
-				(path "/3aef661e-32a5-4098-b535-e9581569514f/20733ad5-b1e0-4da3-932e-70bddfad2269"
+				(path "/244ac675-494c-4e27-8819-02215b480bc3/2561dbd3-5769-4d66-b028-2cb47955e72c"
 					(reference "#PWR075")
 					(unit 1)
@@
 		)
 		(property "Value" "GND"
-			(at 198.12 109.22 0)
-			(hide yes)
-			(effects
-				(font
-					(size 1.0 1.0)
+			(at 198.12 105.62 0)
+			(hide yes)
+			(effects
+				(font
+					(size 1.27 1.27)
 				)
 			)
@@
 		(instances
 			(project "power_board"
-				(path "/3aef661e-32a5-4098-b535-e9581569514f/20733ad5-b1e0-4da3-932e-70bddfad2269"
+				(path "/244ac675-494c-4e27-8819-02215b480bc3/2561dbd3-5769-4d66-b028-2cb47955e72c"
 					(reference "#PWR076")
 					(unit 1)
@@
 		)
 		(property "Value" "GND"
-			(at 177.8 109.22 0)
-			(hide yes)
-			(effects
-				(font
-					(size 1.0 1.0)
+			(at 177.8 105.62 0)
+			(hide yes)
+			(effects
+				(font
+					(size 1.27 1.27)
 				)
 			)
@@
 		(instances
 			(project "power_board"
-				(path "/3aef661e-32a5-4098-b535-e9581569514f/20733ad5-b1e0-4da3-932e-70bddfad2269"
+				(path "/244ac675-494c-4e27-8819-02215b480bc3/2561dbd3-5769-4d66-b028-2cb47955e72c"
 					(reference "#PWR077")
 					(unit 1)
@@
 		)
 		(property "Value" "GND"
-			(at 213.36 118.11 0)
-			(hide yes)
-			(effects
-				(font
-					(size 1.0 1.0)
+			(at 213.36 114.51 0)
+			(hide yes)
+			(effects
+				(font
+					(size 1.27 1.27)
 				)
 			)
@@
 		(instances
 			(project "power_board"
-				(path "/3aef661e-32a5-4098-b535-e9581569514f/20733ad5-b1e0-4da3-932e-70bddfad2269"
+				(path "/244ac675-494c-4e27-8819-02215b480bc3/2561dbd3-5769-4d66-b028-2cb47955e72c"
 					(reference "#PWR078")
 					(unit 1)
@@
 		)
 		(property "Value" "GND"
-			(at 256.54 152.4 0)
-			(hide yes)
-			(effects
-				(font
-					(size 1.0 1.0)
+			(at 256.54 148.8 0)
+			(hide yes)
+			(effects
+				(font
+					(size 1.27 1.27)
 				)
 			)
@@
 		(instances
 			(project "power_board"
-				(path "/3aef661e-32a5-4098-b535-e9581569514f/20733ad5-b1e0-4da3-932e-70bddfad2269"
+				(path "/244ac675-494c-4e27-8819-02215b480bc3/2561dbd3-5769-4d66-b028-2cb47955e72c"
 					(reference "#PWR079")
 					(unit 1)
@@
 		)
 		(property "Value" "+12V"
-			(at 256.54 165.1 0)
-			(hide yes)
-			(effects
-				(font
-					(size 1.0 1.0)
+			(at 256.54 161.5 0)
+			(effects
+				(font
+					(size 1.27 1.27)
 				)
 			)
@@
 		(instances
 			(project "power_board"
-				(path "/3aef661e-32a5-4098-b535-e9581569514f/20733ad5-b1e0-4da3-932e-70bddfad2269"
+				(path "/244ac675-494c-4e27-8819-02215b480bc3/2561dbd3-5769-4d66-b028-2cb47955e72c"
 					(reference "#PWR080")
 					(unit 1)
@@
 		)
 		(property "Value" "GND"
-			(at 256.54 172.72 0)
-			(hide yes)
-			(effects
-				(font
-					(size 1.0 1.0)
+			(at 256.54 169.12 0)
+			(hide yes)
+			(effects
+				(font
+					(size 1.27 1.27)
 				)
 			)
@@
 		(instances
 			(project "power_board"
-				(path "/3aef661e-32a5-4098-b535-e9581569514f/20733ad5-b1e0-4da3-932e-70bddfad2269"
+				(path "/244ac675-494c-4e27-8819-02215b480bc3/2561dbd3-5769-4d66-b028-2cb47955e72c"
 					(reference "#PWR081")
 					(unit 1)
@@
 		)
 		(property "Value" "+5V"
-			(at 256.54 190.5 0)
-			(hide yes)
-			(effects
-				(font
-					(size 1.0 1.0)
+			(at 256.54 186.9 0)
+			(effects
+				(font
+					(size 1.27 1.27)
 				)
 			)
@@
 		(instances
 			(project "power_board"
-				(path "/3aef661e-32a5-4098-b535-e9581569514f/20733ad5-b1e0-4da3-932e-70bddfad2269"
+				(path "/244ac675-494c-4e27-8819-02215b480bc3/2561dbd3-5769-4d66-b028-2cb47955e72c"
 					(reference "#PWR082")
 					(unit 1)
@@
 		)
 		(property "Value" "GND"
-			(at 256.54 203.2 0)
-			(hide yes)
-			(effects
-				(font
-					(size 1.0 1.0)
+			(at 256.54 199.6 0)
+			(hide yes)
+			(effects
+				(font
+					(size 1.27 1.27)
 				)
 			)
@@
 		(instances
 			(project "power_board"
-				(path "/3aef661e-32a5-4098-b535-e9581569514f/20733ad5-b1e0-4da3-932e-70bddfad2269"
+				(path "/244ac675-494c-4e27-8819-02215b480bc3/2561dbd3-5769-4d66-b028-2cb47955e72c"
 					(reference "#PWR083")
 					(unit 1)
@@
 		)
 	)
+	(label "BL_IN"
+		(at 238.76 101.6 0)
+		(effects
+			(font
+				(size 1.27 1.27)
+			)
+			(justify left bottom)
+		)
+	)
 	(label "BOXP_G"
 		(at 107.95 60.96 0)
@@
 		)
 	)
-	(label "BL_IN"
-		(at 238.76 101.6 0)
-		(effects
-			(font
-				(size 1.27 1.27)
-			)
-			(justify left bottom)
-		)
-	)
 	(label "BL_A"
 		(at 196.85 101.6 0)
@@
 	(wire
 		(pts
-			(xy 259.08 101.6)
-			(xy 238.76 101.6)
-		)
-		(stroke
-			(width 0)
-			(type default)
-		)
-	)
-	(wire
-		(pts
 			(xy 238.76 101.6)
 			(xy 237.49 101.6)
 		)
 		(stroke
+			(width 0)
+			(type default)
+		)
+	)
+	(wire
+		(pts
+			(xy 238.76 101.6)
+			(xy 259.08 101.6)
+		)
+		(stroke

Commit message: PCBs routed, labelled and ready to order: Rev 1 fabrication files and buy list
Both boards placed, routed and finished by script (hardware/gen): layout.sh places
(placement.py, with silkscreen names for every terminal, port, header and button),
route.sh routes with Freerouting inside rule areas and net classes from the layout
guide and keeps a board only with 0 DRC errors, 0 unconnected and exact schematic
parity, routespec.sh checks what the DRC cannot (planes, crystal, converter loop,
IPC-2221 widths), finish.sh adds the bottom-silkscreen identification and writes
the fabrication files (gerbers, drill, BOM, positions) only when the DRC passes.

- Pod 70 x 53 mm, 4 layers: In1 solid GND, In2 +3V3, 530 teardrops; no DRC warnings.
- Power 95 x 66 mm, 2 layers, 2 oz: 10 A rail as a zone, converter re-placed (switch
  node 16 mm, feedback 7 mm, no vias; was 78 mm and 40 mm), 328 teardrops.
- Screw terminals turned to open outward; RESET/BOOT side-push on the pod's left
  edge; USB-C footprint with a 3D model (GCT USB4105).
- Pod J2 now the Adafruit 4754's JP1 row pin for pin (the old order shorted its
  3.3 V output to ground); IMU reset on a new J8; HC-05 header fed 5 V.
- Buy list per footprint and module connections in bill-of-materials.md section 10.
- LAYOUT_GUIDE rewritten as how the boards were routed and how to review them;
  decisions, progress log and BUILD_GUIDE updated; power box follows the wider board.
Changed lines of the file:
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@@
 		(instances
 			(project "power_board"
-				(path "/244ac675-494c-4e27-8819-02215b480bc3/2561dbd3-5769-4d66-b028-2cb47955e72c"
+				(path "/c794bf93-11d2-4d5c-a02b-6bb49c306097/cc4a4836-0112-4fbd-b060-cee89dc4dda7"
 					(reference "Q8")
 					(unit 1)
@@
 		(instances
 			(project "power_board"
-				(path "/244ac675-494c-4e27-8819-02215b480bc3/2561dbd3-5769-4d66-b028-2cb47955e72c"
+				(path "/c794bf93-11d2-4d5c-a02b-6bb49c306097/cc4a4836-0112-4fbd-b060-cee89dc4dda7"
 					(reference "R61")
 					(unit 1)
@@
 		(instances
 			(project "power_board"
-				(path "/244ac675-494c-4e27-8819-02215b480bc3/2561dbd3-5769-4d66-b028-2cb47955e72c"
+				(path "/c794bf93-11d2-4d5c-a02b-6bb49c306097/cc4a4836-0112-4fbd-b060-cee89dc4dda7"
 					(reference "R62")
 					(unit 1)
@@
 		(instances
 			(project "power_board"
-				(path "/244ac675-494c-4e27-8819-02215b480bc3/2561dbd3-5769-4d66-b028-2cb47955e72c"
+				(path "/c794bf93-11d2-4d5c-a02b-6bb49c306097/cc4a4836-0112-4fbd-b060-cee89dc4dda7"
 					(reference "J10")
 					(unit 1)
@@
 		(instances
 			(project "power_board"
-				(path "/244ac675-494c-4e27-8819-02215b480bc3/2561dbd3-5769-4d66-b028-2cb47955e72c"
+				(path "/c794bf93-11d2-4d5c-a02b-6bb49c306097/cc4a4836-0112-4fbd-b060-cee89dc4dda7"
 					(reference "R63")
 					(unit 1)
@@
 		(instances
 			(project "power_board"
-				(path "/244ac675-494c-4e27-8819-02215b480bc3/2561dbd3-5769-4d66-b028-2cb47955e72c"
+				(path "/c794bf93-11d2-4d5c-a02b-6bb49c306097/cc4a4836-0112-4fbd-b060-cee89dc4dda7"
 					(reference "U5")
 					(unit 1)
@@
 		(instances
 			(project "power_board"
-				(path "/244ac675-494c-4e27-8819-02215b480bc3/2561dbd3-5769-4d66-b028-2cb47955e72c"
+				(path "/c794bf93-11d2-4d5c-a02b-6bb49c306097/cc4a4836-0112-4fbd-b060-cee89dc4dda7"
 					(reference "D21")
 					(unit 1)
@@
 		(instances
 			(project "power_board"
-				(path "/244ac675-494c-4e27-8819-02215b480bc3/2561dbd3-5769-4d66-b028-2cb47955e72c"
+				(path "/c794bf93-11d2-4d5c-a02b-6bb49c306097/cc4a4836-0112-4fbd-b060-cee89dc4dda7"
 					(reference "J9")
 					(unit 1)
@@
 		(instances
 			(project "power_board"
-				(path "/244ac675-494c-4e27-8819-02215b480bc3/2561dbd3-5769-4d66-b028-2cb47955e72c"
+				(path "/c794bf93-11d2-4d5c-a02b-6bb49c306097/cc4a4836-0112-4fbd-b060-cee89dc4dda7"
 					(reference "J8")
 					(unit 1)
@@
 		(instances
 			(project "power_board"
-				(path "/244ac675-494c-4e27-8819-02215b480bc3/2561dbd3-5769-4d66-b028-2cb47955e72c"
+				(path "/c794bf93-11d2-4d5c-a02b-6bb49c306097/cc4a4836-0112-4fbd-b060-cee89dc4dda7"
 					(reference "J12")
 					(unit 1)
@@
 		(instances
 			(project "power_board"
-				(path "/244ac675-494c-4e27-8819-02215b480bc3/2561dbd3-5769-4d66-b028-2cb47955e72c"
+				(path "/c794bf93-11d2-4d5c-a02b-6bb49c306097/cc4a4836-0112-4fbd-b060-cee89dc4dda7"
 					(reference "#PWR072")
 					(unit 1)
@@
 		(instances
 			(project "power_board"
-				(path "/244ac675-494c-4e27-8819-02215b480bc3/2561dbd3-5769-4d66-b028-2cb47955e72c"
+				(path "/c794bf93-11d2-4d5c-a02b-6bb49c306097/cc4a4836-0112-4fbd-b060-cee89dc4dda7"
 					(reference "#PWR073")
 					(unit 1)
@@
 		(instances
 			(project "power_board"
-				(path "/244ac675-494c-4e27-8819-02215b480bc3/2561dbd3-5769-4d66-b028-2cb47955e72c"
+				(path "/c794bf93-11d2-4d5c-a02b-6bb49c306097/cc4a4836-0112-4fbd-b060-cee89dc4dda7"
 					(reference "#PWR074")
 					(unit 1)
@@
 		(instances
 			(project "power_board"
-				(path "/244ac675-494c-4e27-8819-02215b480bc3/2561dbd3-5769-4d66-b028-2cb47955e72c"
+				(path "/c794bf93-11d2-4d5c-a02b-6bb49c306097/cc4a4836-0112-4fbd-b060-cee89dc4dda7"
 					(reference "#PWR075")
 					(unit 1)
@@
 		(instances
 			(project "power_board"
-				(path "/244ac675-494c-4e27-8819-02215b480bc3/2561dbd3-5769-4d66-b028-2cb47955e72c"
+				(path "/c794bf93-11d2-4d5c-a02b-6bb49c306097/cc4a4836-0112-4fbd-b060-cee89dc4dda7"
 					(reference "#PWR076")
 					(unit 1)
@@
 		(instances
 			(project "power_board"
-				(path "/244ac675-494c-4e27-8819-02215b480bc3/2561dbd3-5769-4d66-b028-2cb47955e72c"
+				(path "/c794bf93-11d2-4d5c-a02b-6bb49c306097/cc4a4836-0112-4fbd-b060-cee89dc4dda7"
 					(reference "#PWR077")
 					(unit 1)
@@
 		(instances
 			(project "power_board"
-				(path "/244ac675-494c-4e27-8819-02215b480bc3/2561dbd3-5769-4d66-b028-2cb47955e72c"
+				(path "/c794bf93-11d2-4d5c-a02b-6bb49c306097/cc4a4836-0112-4fbd-b060-cee89dc4dda7"
 					(reference "#PWR078")
 					(unit 1)
@@
 		(instances
 			(project "power_board"
-				(path "/244ac675-494c-4e27-8819-02215b480bc3/2561dbd3-5769-4d66-b028-2cb47955e72c"
+				(path "/c794bf93-11d2-4d5c-a02b-6bb49c306097/cc4a4836-0112-4fbd-b060-cee89dc4dda7"
 					(reference "#PWR079")
 					(unit 1)
@@
 		(instances
 			(project "power_board"
-				(path "/244ac675-494c-4e27-8819-02215b480bc3/2561dbd3-5769-4d66-b028-2cb47955e72c"
+				(path "/c794bf93-11d2-4d5c-a02b-6bb49c306097/cc4a4836-0112-4fbd-b060-cee89dc4dda7"
 					(reference "#PWR080")
 					(unit 1)
@@
 		(instances
 			(project "power_board"
-				(path "/244ac675-494c-4e27-8819-02215b480bc3/2561dbd3-5769-4d66-b028-2cb47955e72c"
+				(path "/c794bf93-11d2-4d5c-a02b-6bb49c306097/cc4a4836-0112-4fbd-b060-cee89dc4dda7"
 					(reference "#PWR081")
 					(unit 1)
@@
 		(instances
 			(project "power_board"
-				(path "/244ac675-494c-4e27-8819-02215b480bc3/2561dbd3-5769-4d66-b028-2cb47955e72c"
+				(path "/c794bf93-11d2-4d5c-a02b-6bb49c306097/cc4a4836-0112-4fbd-b060-cee89dc4dda7"
 					(reference "#PWR082")
 					(unit 1)
@@
 		(instances
 			(project "power_board"
-				(path "/244ac675-494c-4e27-8819-02215b480bc3/2561dbd3-5769-4d66-b028-2cb47955e72c"
+				(path "/c794bf93-11d2-4d5c-a02b-6bb49c306097/cc4a4836-0112-4fbd-b060-cee89dc4dda7"
 					(reference "#PWR083")
 					(unit 1)
@@
 	(wire
 		(pts
+			(xy 237.49 101.6)
 			(xy 238.76 101.6)
-			(xy 237.49 101.6)
 		)
 		(stroke
@@
 	(wire
 		(pts
+			(xy 106.68 60.96)
+			(xy 107.95 60.96)
+		)
+		(stroke
+			(width 0)
+			(type default)
+		)
+	)
+	(wire
+		(pts
+			(xy 107.95 60.96)
 			(xy 121.92 60.96)
-			(xy 107.95 60.96)
+		)
+		(stroke
+			(width 0)
+			(type default)
+		)
+	)
+	(wire
+		(pts
+			(xy 121.92 57.15)
+			(xy 121.92 60.96)
 		)
 		(stroke
@@
 			(xy 121.92 60.96)
 			(xy 121.92 69.85)
-		)
-		(stroke
-			(width 0)
-			(type default)
-		)
-	)
-	(wire
-		(pts
-			(xy 121.92 57.15)
-			(xy 121.92 60.96)
-		)
-		(stroke
-			(width 0)
-			(type default)
-		)
-	)
-	(wire
-		(pts
-			(xy 106.68 60.96)
-			(xy 107.95 60.96)
 		)
 		(stroke
@@
 	(wire
 		(pts
-			(xy 229.87 101.6)
-			(xy 213.36 101.6)
+			(xy 195.58 101.6)
+			(xy 196.85 101.6)
 		)
 		(stroke
@@
 	(wire
 		(pts
-			(xy 196.85 101.6)
-			(xy 195.58 101.6)
+			(xy 213.36 101.6)
+			(xy 229.87 101.6)
 		)
 		(stroke
@@
 	(wire
 		(pts
+			(xy 30.48 55.88)
+			(xy 31.75 55.88)
+		)
+		(stroke
+			(width 0)
+			(type default)
+		)
+	)
+	(wire
+		(pts
+			(xy 31.75 54.61)
+			(xy 31.75 55.88)
+		)
+		(stroke
+			(width 0)
+			(type default)
+		)
+	)
+	(wire
+		(pts
 			(xy 31.75 54.61)
 			(xy 99.06 54.61)
@@
 	(wire
 		(pts
-			(xy 31.75 54.61)
-			(xy 31.75 55.88)
-		)
-		(stroke
-			(width 0)
-			(type default)
-		)
-	)
-	(wire
-		(pts
 			(xy 99.06 54.61)
 			(xy 99.06 55.88)
@@
 	(wire
 		(pts
-			(xy 30.48 55.88)
-			(xy 31.75 55.88)
-		)
-		(stroke
-			(width 0)
-			(type default)
-		)
-	)
-	(wire
-		(pts
 			(xy 30.48 101.6)
 			(xy 180.34 101.6)
@@
 	(wire
 		(pts
+			(xy 30.48 198.12)
 			(xy 259.08 198.12)
-			(xy 30.48 198.12)
-		)
-		(stroke
-			(width 0)
-			(type default)
-		)
-	)
-	(wire
-		(pts
+		)
+		(stroke
+			(width 0)
+			(type default)
+		)
+	)
+	(wire
+		(pts
+			(xy 30.48 147.32)
 			(xy 259.08 147.32)
-			(xy 30.48 147.32)
-		)
-		(stroke
+		)
+		(stroke

Commit message: Enclosures, brake-light and pod-supply simulations, R63/C1/C2 values, report drafts
Enclosures (hardware/enclosures/): the E-stop housing (yellow ASA box for the 22 mm
mushroom, M16 gland, base to a dash panel), the windscreen pod (rear cover, front shell
whose carrier wall holds board and camera, black front plate with hood, cradle with a
+-8 deg pitch lock on a rail, glass plate template) and the gesture puck (APDS-9960
module under an open window, VHB base). Typical part dimensions are marked VERIFY.
Every STL is a manifold solid.

Simulations: run_brake.sh (PC817 input through the cable to PB5: thresholds with the
weakest and strongest optocoupler, reversed wiring, jump-start, load dump, timing) and
run_pod_supply.sh (cable +5 V and USB diode-OR into the AP2112K: worst cable, lowest
USB, cable pulled while running, USB inrush, back-feed). Both ALL PASS.

Adopted from them, value changes only (copper and teardrops untouched, fab files
regenerated, DRC 0/0, parity exact): power board R63 2.2k -> 4.7k (237 mW in a 24 V
jump-start, beyond the 0805's 125 mW; now 111 mW) and pod C1/C2 10u -> 1u/4.7u (USB
attach inrush 88 uC against USB 2.0's 50 uC; now 28 uC). Order from this commit: the
pcb-rev1.1 tag predates these two changes.

Report: docs/report/final/ drafts Part 16.1 sections 2-6 and 11 from the design as
built, with [RESULT]/[FIGURE]/[CHECK] slots where tests or decisions are pending.
Parts:
- R63: value 2.2k -> 4.7k
Changed lines of the file:
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@@
 			)
 		)
-		(property "Value" "2.2k"
+		(property "Value" "4.7k"
 			(at 233.68 103.866 90)
 			(effects
@@
 			)
 		)
-		(property "Description" "~5 mA LED current at 12 V"
+		(property "Description" "~2.3 mA LED current at 12 V; 4.7k keeps a 24 V jump-start within 0805"
 			(at 233.68 101.6 0)
 			(hide yes)
